Commit message: single robot works on ignition. not sure why controller configs are not loading for >1 robots

File: xarm_description/urdf/common/common.gazebo.xacro (robot description, xacro)
@@ -1,5 +1,5 @@
 <?xml version="1.0"?>
 <robot xmlns:xacro="http://ros.org/wiki/xacro">
-  <xacro:macro name="ignition_ros2_control_plugin" params="prefix:='' ros2_control_params:=''">
+  <xacro:macro name="ignition_ros2_control_plugin" params="prefix:='' namespace:='' ros2_control_params:=''">
     <gazebo>
       <plugin filename="libign_ros2_control-system.so" name="ign_ros2_control::IgnitionROS2ControlPlugin">
@@ -7,5 +7,9 @@
           <parameters>${ros2_control_params}</parameters>
         </xacro:if>
-        <!-- <controller_manager_node_name>${prefix}controller_manager</controller_manager_node_name> -->
+        <xacro:if value="${namespace != ''}">
+          <ros>
+              <namespace>${namespace}</namespace>
+          </ros>
+        </xacro:if>
       </plugin>
     </gazebo>

File: xarm_description/urdf/xarm_device_macro.xacro (robot description, xacro)
@@ -276,5 +276,5 @@
         </xacro:if>
         <xacro:if value="${ros2_control_plugin == 'ign_ros2_control/IgnitionSystem'}">
-          <xacro:ignition_ros2_control_plugin prefix="${prefix}" ros2_control_params="${new_ros2_control_params}"/>
+          <xacro:ignition_ros2_control_plugin prefix="${prefix}" namespace="${hw_ns}" ros2_control_params="${new_ros2_control_params}"/>
         </xacro:if>
         <xacro:unless value="${ros2_control_plugin == 'ign_ros2_control/IgnitionSystem'}">
