Commit message: Finished the xArm6 MPPI-Isaac integration

File: xarm_description/urdf/common/common.link.xacro (robot description, xacro)
@@ -38,5 +38,5 @@
     </visual>
   </xacro:macro>
-  <xacro:macro name="common_link_collision" params="mesh_filename add_mesh_suffix:=true origin_xyz:='0 0 0' origin_rpy:='0 0 0'">
+  <xacro:macro name="common_link_collision" params="mesh_filename add_mesh_suffix:=true other_mesh_suffix:='stl' origin_xyz:='0 0 0' origin_rpy:='0 0 0'">
     <collision>
       <geometry>
@@ -45,5 +45,5 @@
         </xacro:if>
         <xacro:unless value="${add_mesh_suffix}">
-          <mesh filename="${mesh_path}/${mesh_filename}"/>
+          <mesh filename="${mesh_path}/${mesh_filename}.${other_mesh_suffix}"/>
         </xacro:unless>
       </geometry>
@@ -54,5 +54,5 @@
     <origin xyz="${joint_kinematic_params['x']} ${joint_kinematic_params['y']} ${joint_kinematic_params['z']}" rpy="${joint_kinematic_params['roll']} ${joint_kinematic_params['pitch']} ${joint_kinematic_params['yaw']}" />
   </xacro:macro>
-  <xacro:macro name="parse_link_inertial_filename" params="dof robot_type robot_sn model1300">
+  <xacro:macro name="parse_link_inertial_filename" params="dof robot_type robot_sn model_num">
     <!-- default inertial params filename -->
     <xacro:property name="inertial_params_filename" value="xarm${dof}_type${dof}_HT_BR2"/>
@@ -75,5 +75,5 @@
     <xacro:property name="mass_type" value="-1" />
     <xacro:property name="model_type" value="-1" />
-    <xacro:property name="_model1300" value="${model1300}" />
+    <xacro:property name="_model1300" value="${model_num >= 1300}" />
     <!-- parse model_type and mass_type from robot_sn -->
     <xacro:if value="${robot_sn_len >= 14 and (robot_sn[0] == 'X' or robot_sn[0] == 'L' or robot_sn[0] == 'F')}">

File: xarm_description/urdf/xarm6/xarm6.gazebo.xacro (robot description, xacro)
@@ -23,4 +23,8 @@
       <selfCollide>true</selfCollide>
     </gazebo>
+    <!-- End effector tip measurement tools -->
+    <!-- <gazebo reference="${prefix}ee_tip">
+      <selfCollide>true</selfCollide>
+    </gazebo> -->
   </xacro:macro>
 </robot>

File: xarm_description/urdf/xarm6/xarm6.ros2_control.xacro (robot description, xacro)
@@ -6,10 +6,10 @@
     hw_ns:='xarm' add_gripper:='false' add_bio_gripper:='false'
     robot_ip:='' report_type:='normal' baud_checkset:='true' default_gripper_baud:=2000000
-    joint1_lower_limit:=${-2.0*pi}  joint1_upper_limit:=${2.0*pi}
-    joint2_lower_limit:=${-2.059}  joint2_upper_limit:=${2.0944}
-    joint3_lower_limit:=${-3.927}  joint3_upper_limit:=${0.19198}
-    joint4_lower_limit:=${-2.0*pi}  joint4_upper_limit:=${2.0*pi}
-    joint5_lower_limit:=${-1.69297}  joint5_upper_limit:=${pi}
-    joint6_lower_limit:=${-2.0*pi}  joint6_upper_limit:=${2.0*pi}">
+    joint1_lower_limit:=${-10*pi}  joint1_upper_limit:=${10*pi}
+    joint2_lower_limit:=${-10*pi}  joint2_upper_limit:=${10*pi}
+    joint3_lower_limit:=${-10*pi}  joint3_upper_limit:=${10*pi}
+    joint4_lower_limit:=${-10*pi}  joint4_upper_limit:=${10*pi}
+    joint5_lower_limit:=${-10*pi}  joint5_upper_limit:=${10*pi}
+    joint6_lower_limit:=${-10*pi}  joint6_upper_limit:=${10*pi}">
     <ros2_control name="${prefix}${ros2_control_plugin}" type="system">
       <hardware>

File: xarm_description/urdf/xarm6/xarm6.urdf.xacro (robot description, xacro)
@@ -2,21 +2,35 @@
 <robot xmlns:xacro="http://ros.org/wiki/xacro">
   <xacro:macro name="xarm6_urdf" params="prefix
-    joint1_lower_limit:=${-2.0*pi}  joint1_upper_limit:=${2.0*pi}
-    joint2_lower_limit:=${-2.059}  joint2_upper_limit:=${2.0944}
-    joint3_lower_limit:=${-3.927}  joint3_upper_limit:=${0.19198}
-    joint4_lower_limit:=${-2.0*pi}  joint4_upper_limit:=${2.0*pi}
-    joint5_lower_limit:=${-1.69297}  joint5_upper_limit:=${pi}
-    joint6_lower_limit:=${-2.0*pi}  joint6_upper_limit:=${2.0*pi}
-    model1300:=false
+    joint1_lower_limit:=${-10.0*pi}  joint1_upper_limit:=${10.0*pi}
+    joint2_lower_limit:=${-10*pi}  joint2_upper_limit:=${10*pi}
+    joint3_lower_limit:=${-10*pi}  joint3_upper_limit:=${10*pi}
+    joint4_lower_limit:=${-10*pi}  joint4_upper_limit:=${10*pi}
+    joint5_lower_limit:=${-10*pi}  joint5_upper_limit:=${10*pi}
+    joint6_lower_limit:=${-10*pi}  joint6_upper_limit:=${10*pi}
+    model_num:=0
     inertial_params_filename:='' kinematics_params_filename:='' "
     >
     <!-- define property -->
-    <xacro:if value="${model1300}">
-      <xacro:property name="end_tool_visual_filename" value="end_tool/visual/end_tool_1300"/>
-      <xacro:property name="end_tool_collision_filename" value="end_tool/collision/end_tool_1300"/>
+    <xacro:if value="${model_num >= 1305 and model_num != 1380}">
+      <xacro:property name="visual_dir" value="xarm6_1305/visual"/>
+      <xacro:property name="collision_dir" value="xarm6_1305/collision"/>
+      <xacro:property name="add_mesh_suffix" value="false"/>
+      <xacro:property name="collison_mesh_suffix" value="obj"/>
+      <xacro:property name="link6_visual" value="xarm6_1305/visual/link6"/>
+      <xacro:property name="link6_collision" value="xarm6_1305/collision/link6"/>
     </xacro:if>
-    <xacro:unless value="${model1300}">
-      <xacro:property name="end_tool_visual_filename" value="xarm6/visual/link6"/>
-      <xacro:property name="end_tool_collision_filename" value="end_tool/collision/end_tool"/>
+    <xacro:unless value="${model_num >= 1305 and model_num != 1380}">
+      <xacro:property name="visual_dir" value="xarm6/visual"/>
+      <xacro:property name="collision_dir" value="xarm6/visual"/>
+      <xacro:property name="add_mesh_suffix" value="true"/>
+      <xacro:property name="collison_mesh_suffix" value="stl"/>
+      <xacro:if value="${model_num >= 1300}">
+        <xacro:property name="link6_visual" value="end_tool/visual/end_tool_1300"/>
+        <xacro:property name="link6_collision" value="end_tool/collision/end_tool_1300"/>
+      </xacro:if>
+      <xacro:unless value="${model_num >= 1300}">
+        <xacro:property name="link6_visual" value="xarm6/visual/link6"/>
+        <xacro:property name="link6_collision" value="end_tool/collision/end_tool"/>
+      </xacro:unless>
     </xacro:unless>
     <!-- load params and define property -->
@@ -46,10 +60,12 @@
       </inertial>
       <xacro:common_link_visual
-        mesh_filename="xarm6/visual/link_base"
-        origin_xyz="0 0 0"
-        origin_rpy="0 0 0"
-        material_name="${prefix}White" />
-      <xacro:common_link_collision
-        mesh_filename="xarm6/visual/link_base"
+        mesh_filename="${visual_dir}/link_base"
+        origin_xyz="0 0 0"
+        origin_rpy="0 0 0"
+        material_name="${prefix}White" />
+      <xacro:common_link_collision
+        mesh_filename="${collision_dir}/link_base"
+        add_mesh_suffix="${add_mesh_suffix}"
+        other_mesh_suffix="${collison_mesh_suffix}"
         origin_xyz="0 0 0"
         origin_rpy="0 0 0" />
@@ -60,10 +76,12 @@
         origin_rpy="0 0 0"/>
       <xacro:common_link_visual
-        mesh_filename="xarm6/visual/link1"
-        origin_xyz="0 0 0"
-        origin_rpy="0 0 0"
-        material_name="${prefix}White" />
-      <xacro:common_link_collision
-        mesh_filename="xarm6/visual/link1"
+        mesh_filename="${visual_dir}/link1"
+        origin_xyz="0 0 0"
+        origin_rpy="0 0 0"
+        material_name="${prefix}White" />
+      <xacro:common_link_collision
+        mesh_filename="${collision_dir}/link1"
+        add_mesh_suffix="${add_mesh_suffix}"
+        other_mesh_suffix="${collison_mesh_suffix}"
         origin_xyz="0 0 0"
         origin_rpy="0 0 0" />
@@ -81,4 +99,5 @@
         velocity="3.14"/>
       <dynamics damping="1.0" friction="1.0"/>
+      <initial_position>0.0</initial_position>
     </joint>
     <link name="${prefix}link2">
@@ -87,11 +106,13 @@
         origin_rpy="0 0 0"/>
       <xacro:common_link_visual
-        mesh_filename="xarm6/visual/link2"
-        origin_xyz="0 0 ${-kinematics_params['joint2']['y']}"
-        origin_rpy="0 0 0"
-        material_name="${prefix}White" />
-      <xacro:common_link_collision
-        mesh_filename="xarm6/visual/link2"
-        origin_xyz="0 0 ${-kinematics_params['joint2']['y']}"
+        mesh_filename="${visual_dir}/link2"
+        origin_xyz="0 0 0"
+        origin_rpy="0 0 0"
+        material_name="${prefix}White" />
+      <xacro:common_link_collision
+        mesh_filename="${collision_dir}/link2"
+        add_mesh_suffix="${add_mesh_suffix}"
+        other_mesh_suffix="${collison_mesh_suffix}"
+        origin_xyz="0 0 0"
         origin_rpy="0 0 0" />
     </link>
@@ -99,5 +120,5 @@
       <parent link="${prefix}link1"/>
       <child link="${prefix}link2"/>
-      <origin xyz="0 0 0" rpy="-1.5708 -0.5 0" />
+      <!-- <origin xyz="0 0 0" rpy="-1.5708 0 0" /> -->
       <xacro:common_joint_origin joint_kinematic_params="${kinematics_params['joint2']}" />
       <axis xyz="0 0 1"/>
@@ -108,4 +129,5 @@
         velocity="3.14"/>
       <dynamics damping="1.0" friction="1.0"/>
+      <initial_position>-0.78</initial_position>
     </joint>
     <link name="${prefix}link3">
@@ -114,10 +136,12 @@
         origin_rpy="0 0 0"/>
       <xacro:common_link_visual
-        mesh_filename="xarm6/visual/link3"
-        origin_xyz="0 0 0"
-        origin_rpy="0 0 0"
-        material_name="${prefix}White" />
-      <xacro:common_link_collision
-        mesh_filename="xarm6/visual/link3"
+        mesh_filename="${visual_dir}/link3"
+        origin_xyz="0 0 0"
+        origin_rpy="0 0 0"
+        material_name="${prefix}White" />
+      <xacro:common_link_collision
+        mesh_filename="${collision_dir}/link3"
+        add_mesh_suffix="${add_mesh_suffix}"
+        other_mesh_suffix="${collison_mesh_suffix}"
         origin_xyz="0 0 0"
         origin_rpy="0 0 0" />
@@ -126,5 +150,5 @@
       <parent link="${prefix}link2"/>
       <child link="${prefix}link3"/>
-      <origin xyz="0.0535 -0.2845 0" rpy="0 0 -0.5"/>
+      <!-- <origin xyz="0.0535 -0.2845 0" rpy="0 0 0"/> -->
       <xacro:common_joint_origin joint_kinematic_params="${kinematics_params['joint3']}" />
       <axis xyz="0 0 1"/>
@@ -135,4 +159,5 @@
         velocity="3.14"/>
       <dynamics damping="1.0" friction="1.0"/>
+      <initial_position>-0.78</initial_position>
     </joint>
     <link name="${prefix}link4">
@@ -141,10 +166,12 @@
         origin_rpy="0 0 0"/>
       <xacro:common_link_visual
-        mesh_filename="xarm6/visual/link4"
-        origin_xyz="0 0 0"
-        origin_rpy="0 0 0"
-        material_name="${prefix}White" />
-      <xacro:common_link_collision
-        mesh_filename="xarm6/visual/link4"
+        mesh_filename="${visual_dir}/link4"
+        origin_xyz="0 0 0"
+        origin_rpy="0 0 0"
+        material_name="${prefix}White" />
+      <xacro:common_link_collision
+        mesh_filename="${collision_dir}/link4"
+        add_mesh_suffix="${add_mesh_suffix}"
+        other_mesh_suffix="${collison_mesh_suffix}"
         origin_xyz="0 0 0"
         origin_rpy="0 0 0" />
@@ -162,4 +189,5 @@
         velocity="3.14"/>
       <dynamics damping="1.0" friction="1.0"/>
+      <initial_position>0.0</initial_position>
     </joint>
     <link name="${prefix}link5">
@@ -168,10 +196,12 @@
         origin_rpy="0 0 0"/>
       <xacro:common_link_visual
-        mesh_filename="xarm6/visual/link5"
-        origin_xyz="0 0 0"
-        origin_rpy="0 0 0"
-        material_name="${prefix}White" />
-      <xacro:common_link_collision
-        mesh_filename="xarm6/visual/link5"
+        mesh_filename="${visual_dir}/link5"
+        origin_xyz="0 0 0"
+        origin_rpy="0 0 0"
+        material_name="${prefix}White" />
+      <xacro:common_link_collision
+        mesh_filename="${collision_dir}/link5"
+        add_mesh_suffix="${add_mesh_suffix}"
+        other_mesh_suffix="${collison_mesh_suffix}"
         origin_xyz="0 0 0"
         origin_rpy="0 0 0" />
@@ -180,5 +210,4 @@
       <parent link="${prefix}link4"/>
       <child link="${prefix}link5"/>
-      <origin xyz="0.0 0.0 0.0" rpy="1.5708 -0.95 0.0"/>
       <xacro:common_joint_origin joint_kinematic_params="${kinematics_params['joint5']}" />
       <axis xyz="0 0 1"/>
@@ -189,4 +218,5 @@
         velocity="3.14"/>
       <dynamics damping="1.0" friction="1.0"/>
+      <initial_position>1.5708</initial_position>
     </joint>
     <link name="${prefix}link6">
@@ -195,10 +225,12 @@
         origin_rpy="0 0 0"/>
       <xacro:common_link_visual
-        mesh_filename="${end_tool_visual_filename}"
+        mesh_filename="${link6_visual}"
         origin_xyz="0 0 0"
         origin_rpy="0 0 0"
         material_name="${prefix}Silver" />
       <xacro:common_link_collision
-        mesh_filename="${end_tool_collision_filename}"
+        mesh_filename="${link6_collision}"
+        add_mesh_suffix="${add_mesh_suffix}"
+        other_mesh_suffix="${collison_mesh_suffix}"
         origin_xyz="0 0 0"
         origin_rpy="0 0 0" />
@@ -216,5 +248,100 @@
         velocity="3.14"/>
       <dynamics damping="1.0" friction="1.0"/>
-    </joint>
+      <initial_position>0.0</initial_position>
+    </joint>
+  <link name="${prefix}ee_stick">
+    <visual>
+      <geometry>
+        <cylinder length="0.35" radius="0.01"/>
+      </geometry>
+      <origin rpy="0 0 0" xyz="0 0 0.16"/>
+      <material name="Purple">
+        <color rgba="0.5 0 0.5 1"/>
+      </material>
+    </visual>
+    <collision>
+      <geometry>
+        <cylinder length="0.35" radius="0.01"/>
+      </geometry>
+      <origin rpy="0 0 0" xyz="0 0 0.16"/>
+    </collision>
+  </link>
+  <joint name="${prefix}joint_ee_stick" type="fixed">
+    <origin rpy="0 0 0" xyz="0 0 -0.015"/>
+    <parent link="${prefix}link6"/>
+    <child link="${prefix}ee_stick"/>
+    <axis xyz="0 0 0"/>
+  </joint>
+  <link name="${prefix}ee_tip">
+    <!-- Visual marker for end effector tip -->
+    <visual>
+      <origin xyz="0 0 0" rpy="0 0 0"/>
+      <geometry>
+        <sphere radius="0.01"/>
+      </geometry>
+      <material name="red">
+        <color rgba="1 0 0 1"/>
+      </material>
+    </visual>
+    <!-- Coordinate frame visualization -->
+    <visual>
+      <origin xyz="0 0 0" rpy="0 0 0"/>
+      <geometry>
+        <cylinder radius="0.002" length="0.05"/>
+      </geometry>
+      <material name="blue">
+        <color rgba="0 0 1 1"/>
+      </material>
+    </visual>
+    <!-- X-axis marker -->
+    <visual>
+      <origin xyz="0.025 0 0" rpy="0 0 0"/>
+      <geometry>
+        <cylinder radius="0.001" length="0.05"/>
+      </geometry>
+      <material name="green">
+        <color rgba="0 1 0 1"/>
+      </material>
+    </visual>
+    <!-- Y-axis marker -->
+    <visual>
+      <origin xyz="0 0.025 0" rpy="0 0 1.5708"/>
+      <geometry>
+        <cylinder radius="0.001" length="0.05"/>
+      </geometry>
+      <material name="yellow">
+        <color rgba="1 1 0 1"/>
+      </material>
+    </visual>
+    <!-- Z-axis marker -->
+    <visual>
+      <origin xyz="0 0 0.025" rpy="0 -1.5708 0"/>
+      <geometry>
+        <cylinder radius="0.001" length="0.05"/>
+      </geometry>
+      <material name="magenta">
+        <color rgba="1 0 1 1"/>
+      </material>
+    </visual>
+    <!-- Collision geometry for end effector tip -->
+    <collision>
+      <origin xyz="0 0 0" rpy="0 0 0"/>
+      <geometry>
+        <sphere radius="0.01"/>
+      </geometry>
+    </collision>
+    <!-- Inertial properties -->
+    <inertial>
+      <origin xyz="0 0 0" rpy="0 0 0"/>
+      <mass value="0.001"/>
+      <inertia ixx="0.000001" ixy="0" ixz="0" iyy="0.000001" iyz="0" izz="0.000001"/>
+    </inertial>
+  </link>
+  <joint name="${prefix}joint_ee_tip" type="fixed">
+    <origin rpy="0 0 0" xyz="0 0 0.335"/>
+    <parent link="${prefix}ee_stick"/>
+    <child link="${prefix}ee_tip"/>
+    <axis xyz="0 0 0"/>
+  </joint>
     <!-- <link name="${prefix}link_eef" />
     <joint name="${prefix}joint_eef" type="fixed">

File: xarm_description/urdf/xarm_device.urdf.xacro (robot description, xacro)
@@ -58,5 +58,5 @@
     baud_checkset="${robot_spec['baud_checkset']}"
     default_gripper_baud="${robot_spec['default_gripper_baud']}"
-    model1300="${robot_spec['model1300']}"
+    model_num="${robot_spec['model_num']}"
     robot_sn="${robot_spec['robot_sn']}"
     limited="${robot_spec['limited']}"

File: xarm_description/urdf/xarm_device_macro.xacro (robot description, xacro)
@@ -37,5 +37,5 @@
     baud_checkset:=true
     default_gripper_baud:=2000000
-    model1300:=false
+    model_num:=0
     robot_sn:=''
     mesh_suffix:='stl'
@@ -60,7 +60,7 @@
     <!-- include common.link.xacro -->
     <xacro:include filename="$(find xarm_description)/urdf/common/common.link.xacro" />
-    <xacro:parse_link_inertial_filename dof="${dof}" robot_type="${robot_type}" robot_sn="${robot_sn}" model1300="${model1300}" />
+    <xacro:parse_link_inertial_filename dof="${dof}" robot_type="${robot_type}" robot_sn="${robot_sn}" model_num="${model_num}" />
     <xacro:property name="inertial_params_filename" value="${scope_parent_inertial_params_filename}"/>
-    <xacro:property name="new_model1300" value="${scope_parent_model1300}"/>
+    <xacro:property name="new_model_num" value="${scope_parent_model_num}"/>
     <!-- add one world link if no 'attach_to' specified  -->
     <xacro:if value="${attach_to != ''}">
@@ -127,5 +127,5 @@
           baud_checkset="${baud_checkset}"
           default_gripper_baud="${default_gripper_baud}"
-          model1300="${new_model1300}"
+          model_num="${new_model_num}"
           inertial_params_filename="${inertial_params_filename}"
           kinematics_params_filename="${kinematics_params_filename}"
@@ -159,5 +159,5 @@
           baud_checkset="${baud_checkset}"
           default_gripper_baud="${default_gripper_baud}"
-          model1300="${new_model1300}"
+          model_num="${model_num}"
           inertial_params_filename="${inertial_params_filename}"
           kinematics_params_filename="${kinematics_params_filename}"
@@ -178,5 +178,5 @@
           baud_checkset="${baud_checkset}"
           default_gripper_baud="${default_gripper_baud}"
-          model1300="${new_model1300}"
+          model_num="${new_model_num}"
           inertial_params_filename="${inertial_params_filename}"
           kinematics_params_filename="${kinematics_params_filename}"
@@ -195,5 +195,5 @@
           baud_checkset="${baud_checkset}"
           default_gripper_baud="${default_gripper_baud}"
-          model1300="${new_model1300}"
+          model_num="${new_model_num}"
           inertial_params_filename="${inertial_params_filename}"
           kinematics_params_filename="${kinematics_params_filename}"
