Commit message: load gazebo plugins by default. dont worry about other geometry..

File: xarm_description/urdf/dual_xarm_device.urdf.xacro (robot description, xacro)
@@ -69,5 +69,5 @@
     add_bio_gripper="$(arg add_bio_gripper_1)" dof="$(arg dof_1)"
     ros2_control_plugin="$(arg ros2_control_plugin)" robot_type="$(arg robot_type_1)"
-    load_gazebo_plugin="false" ros2_control_params="$(arg ros2_control_params)"
+    ros2_control_params="$(arg ros2_control_params)"
     attach_to="world" attach_xyz="0 0 0" attach_rpy="0 0 0"
     add_realsense_d435i="$(arg add_realsense_d435i_1)"
@@ -88,5 +88,5 @@
     add_bio_gripper="$(arg add_bio_gripper_2)" dof="$(arg dof_2)"
     ros2_control_plugin="$(arg ros2_control_plugin)" robot_type="$(arg robot_type_2)"
-    load_gazebo_plugin="true" ros2_control_params="$(arg ros2_control_params)"
+    ros2_control_params="$(arg ros2_control_params)"
     attach_to="world" attach_xyz="0 1 0" attach_rpy="0 0 0" create_attach_link="false"
     add_realsense_d435i="$(arg add_realsense_d435i_2)"

File: xarm_description/urdf/xarm_device.urdf.xacro (robot description, xacro)
@@ -46,5 +46,5 @@
     add_bio_gripper="$(arg add_bio_gripper)" dof="$(arg dof)"
     ros2_control_plugin="$(arg ros2_control_plugin)" robot_type="$(arg robot_type)"
-    load_gazebo_plugin="true" ros2_control_params="$(arg ros2_control_params)"
+    ros2_control_params="$(arg ros2_control_params)"
     add_realsense_d435i="$(arg add_realsense_d435i)"
     add_d435i_links="$(arg add_d435i_links)"

File: xarm_description/urdf/xarm_device_macro.xacro (robot description, xacro)
@@ -18,5 +18,4 @@
     create_attach_link:=true
     ros2_control_params:=''
-    load_gazebo_plugin:=false
     add_realsense_d435i:=false
     add_d435i_links:=true
@@ -200,4 +199,5 @@
       </xacro:unless>
     </xacro:unless>
+    <!-- Grippers and end effectors -->
     <xacro:if value="${add_realsense_d435i}">
       <!-- (xarm) Load RealSense D435i URDF -->
@@ -263,27 +263,20 @@
     </xacro:if>
     <!-- gazebo_plugin -->
-    <xacro:if value="${load_gazebo_plugin}">
-      <xacro:include filename="$(find xarm_description)/urdf/common/common.gazebo.xacro" />
-      <xacro:if value="${is_ros2}">
-        <xacro:if value="${robot_type == 'uf850' or robot_type == 'xarm7_mirror'}">
-          <xacro:property name="new_ros2_control_params" value="$(find xarm_controller)/config/${robot_type}_controllers.yaml"/>
-        </xacro:if>
-        <xacro:unless value="${robot_type == 'uf850' or robot_type == 'xarm7_mirror'}">
-          <xacro:property name="new_ros2_control_params" value="$(find xarm_controller)/config/${robot_type}${dof}_controllers.yaml"/>
-        </xacro:unless>
-        <xacro:if value="${ros2_control_params != ''}">
-          <xacro:property name="new_ros2_control_params" value="${ros2_control_params}"/>
-        </xacro:if>
-        <xacro:if value="${ros2_control_plugin == 'ign_ros2_control/IgnitionSystem'}">
-          <xacro:ignition_ros2_control_plugin prefix="${prefix}" namespace="${hw_ns}" ros2_control_params="${new_ros2_control_params}"/>
-        </xacro:if>
-        <xacro:unless value="${ros2_control_plugin == 'ign_ros2_control/IgnitionSystem'}">
-          <xacro:gazebo_ros2_control_plugin ros2_control_params="${new_ros2_control_params}"/>
-        </xacro:unless>
-      </xacro:if>
-      <xacro:unless value="${is_ros2}">
-        <xacro:gazebo_ros1_control_plugin namespace="${hw_ns}"/>
-      </xacro:unless>
-    </xacro:if>
+    <!-- no harm in loading gazebo tags. just let them load -->
+    <xacro:include filename="$(find xarm_description)/urdf/common/common.gazebo.xacro" />
+    <!-- If not overriden, use default controller configs -->
+    <xacro:if value="${ros2_control_params != ''}">
+      <xacro:property name="new_ros2_control_params" value="${ros2_control_params}"/>
+    </xacro:if>
+    <xacro:unless value="${ros2_control_params != ''}">
+      <xacro:property name="new_ros2_control_params" value="${find xarm_controller/config/${robot_name}_controllers.yaml}" />
+    </xacro:unless>
+    <!-- Detect whether to use ignition or classic -->
+    <xacro:if value="${ros2_control_plugin == 'ign_ros2_control/IgnitionSystem'}">
+      <xacro:ignition_ros2_control_plugin prefix="${prefix}" namespace="${hw_ns}" ros2_control_params="${new_ros2_control_params}"/>
+    </xacro:if>
+    <xacro:unless value="${ros2_control_plugin == 'ign_ros2_control/IgnitionSystem'}">
+      <xacro:gazebo_ros2_control_plugin ros2_control_params="${new_ros2_control_params}"/>
+    </xacro:unless>
     <xacro:if value="${use_gazebo_camera}">
       <xacro:include filename="$(find xarm_description)/urdf/camera/camera.gazebo.xacro" />
