Commit message: move other geometry to a yaml file

File: xarm_description/urdf/xarm_device.urdf.xacro (robot description, xacro)
@@ -20,16 +20,11 @@
   <xacro:arg name="add_d435i_links" default="true"/>
   <xacro:arg name="use_gazebo_camera" default="false"/>
-  <xacro:arg name="add_other_geometry" default="false"/>
-  <xacro:arg name="geometry_type" default="box"/>
-  <xacro:arg name="geometry_mass" default="0.1"/>
-  <xacro:arg name="geometry_height" default="0.1"/>
-  <xacro:arg name="geometry_radius" default="0.1"/>
-  <xacro:arg name="geometry_length" default="0.1"/>
-  <xacro:arg name="geometry_width" default="0.1"/>
-  <xacro:arg name="geometry_mesh_filename" default=""/>
-  <xacro:arg name="geometry_mesh_origin_xyz" default="0 0 0"/>
-  <xacro:arg name="geometry_mesh_origin_rpy" default="0 0 0"/>
-  <xacro:arg name="geometry_mesh_tcp_xyz" default="0 0 0"/>
-  <xacro:arg name="geometry_mesh_tcp_rpy" default="0 0 0"/>
+  <xacro:arg name="other_geometry_config_file"
+    default="$(find xarm_description)/config/default_urdf_arguments/other_geometry.yaml"
+  />
+  <xacro:property name="other_geometry_config_file" value="$(arg other_geometry_config_file)" />
+  <xacro:property name="other_geometry"
+    value="${xacro.load_yaml(other_geometry_config_file)}"
+  />
   <xacro:arg name="baud_checkset" default="true"/>
   <xacro:arg name="default_gripper_baud" default="2000000"/>
@@ -41,22 +36,44 @@
   <!-- load xarm device -->
   <xacro:include filename="$(find xarm_description)/urdf/xarm_device_macro.xacro" />
-  <xacro:xarm_device prefix="$(arg prefix)" hw_ns="$(arg hw_ns)" limited="$(arg limited)"
-    effort_control="$(arg effort_control)" velocity_control="$(arg velocity_control)"
-    add_gripper="$(arg add_gripper)" add_vacuum_gripper="$(arg add_vacuum_gripper)"
-    add_bio_gripper="$(arg add_bio_gripper)" dof="$(arg dof)"
-    ros2_control_plugin="$(arg ros2_control_plugin)" robot_type="$(arg robot_type)"
+  <!-- TODO: maybe make the macros use dicts themselves, but that might be digging too deep -->
+  <xacro:xarm_device
+    prefix="$(arg prefix)"
+    hw_ns="$(arg hw_ns)"
+    ros2_control_plugin="$(arg ros2_control_plugin)"
     ros2_control_params="$(arg ros2_control_params)"
+    robot_ip="$(arg robot_ip)"
+    dof="$(arg dof)"
+    robot_type="$(arg robot_type)"
+    report_type="$(arg report_type)"
+    baud_checkset="$(arg baud_checkset)"
+    default_gripper_baud="$(arg default_gripper_baud)"
+    model1300="$(arg model1300)"
+    robot_sn="$(arg robot_sn)"
+    limited="$(arg limited)"
+    effort_control="$(arg effort_control)"
+    velocity_control="$(arg velocity_control)"
+    attach_to="$(arg attach_to)"
+    attach_xyz="$(arg attach_xyz)"
+    attach_rpy="$(arg attach_rpy)"
+    add_gripper="$(arg add_gripper)"
+    add_vacuum_gripper="$(arg add_vacuum_gripper)"
+    add_bio_gripper="$(arg add_bio_gripper)"
     add_realsense_d435i="$(arg add_realsense_d435i)"
     add_d435i_links="$(arg add_d435i_links)"
-    add_other_geometry="$(arg add_other_geometry)"
-    geometry_type="$(arg geometry_type)" geometry_mass="$(arg geometry_mass)"
-    geometry_height="$(arg geometry_height)" geometry_radius="$(arg geometry_radius)"
-    geometry_length="$(arg geometry_length)" geometry_width="$(arg geometry_width)"
-    geometry_mesh_filename="$(arg geometry_mesh_filename)"
-    geometry_mesh_origin_xyz="$(arg geometry_mesh_origin_xyz)" geometry_mesh_origin_rpy="$(arg geometry_mesh_origin_rpy)"
-    geometry_mesh_tcp_xyz="$(arg geometry_mesh_tcp_xyz)" geometry_mesh_tcp_rpy="$(arg geometry_mesh_tcp_rpy)"
-    robot_ip="$(arg robot_ip)" report_type="$(arg report_type)"
-    baud_checkset="$(arg baud_checkset)" default_gripper_baud="$(arg default_gripper_baud)"
-    model1300="$(arg model1300)" attach_to="$(arg attach_to)" attach_xyz="$(arg attach_xyz)" attach_rpy="$(arg attach_rpy)"
-    robot_sn="$(arg robot_sn)" use_gazebo_camera="$(arg use_gazebo_camera)" mesh_suffix="$(arg mesh_suffix)" kinematics_suffix="$(arg kinematics_suffix)" />
+    mesh_suffix="$(arg mesh_suffix)"
+    kinematics_suffix="$(arg kinematics_suffix)"
+    use_gazebo_camera="$(arg use_gazebo_camera)"
+    add_other_geometry="${other_geometry['add']}"
+    geometry_type="${other_geometry['type']}"
+    geometry_mass="${other_geometry['mass']}"
+    geometry_height="${other_geometry['height']}"
+    geometry_radius="${other_geometry['radius']}"
+    geometry_length="${other_geometry['length']}"
+    geometry_width="${other_geometry['width']}"
+    geometry_mesh_filename="${other_geometry['mesh_filename']}"
+    geometry_mesh_origin_xyz="${other_geometry['mesh_origin_xyz']}"
+    geometry_mesh_origin_rpy="${other_geometry['mesh_origin_rpy']}"
+    geometry_mesh_tcp_xyz="${other_geometry['mesh_tcp_xyz']}"
+    geometry_mesh_tcp_rpy="${other_geometry['mesh_tcp_rpy']}"
+  />
 </robot>

Commit message: make unnecessary params come from yaml

File: xarm_description/urdf/xarm_device.urdf.xacro (robot description, xacro)
@@ -1,37 +1,47 @@
 <?xml version='1.0' encoding='utf-8'?>
 <robot xmlns:xacro="http://ros.org/wiki/xacro" name="UF_ROBOT">
+  <!-- macro for having property with the same name/value as an argument -->
+  <xacro:macro name="define_arg_property" params="prop_name default">
+    <xacro:arg name="${prop_name}" default="${default}"/>
+    <xacro:property name="${prop_name}" value="$(arg ${prop_name})"/>
+  </xacro:macro>
   <xacro:arg name="prefix" default=""/>
   <xacro:arg name="hw_ns" default="xarm"/>
-  <xacro:arg name="limited" default="false"/>
-  <xacro:arg name="effort_control" default="false"/>
-  <xacro:arg name="velocity_control" default="false"/>
-  <xacro:arg name="add_gripper" default="false"/>
-  <xacro:arg name="add_vacuum_gripper" default="false"/>
-  <xacro:arg name="add_bio_gripper" default="false"/>
-  <xacro:arg name="model1300" default="false"/>
-  <xacro:arg name="dof" default="7"/>
-  <xacro:arg name="robot_ip" default=""/>
-  <xacro:arg name="robot_type" default="xarm"/>
-  <xacro:arg name="robot_sn" default=""/>
-  <xacro:arg name="report_type" default="normal"/>
   <xacro:arg name="ros2_control_plugin" default="uf_robot_hardware/UFRobotSystemHardware"/>
   <xacro:arg name="ros2_control_params" default=""/>
-  <xacro:arg name="add_realsense_d435i" default="false"/>
-  <xacro:arg name="add_d435i_links" default="true"/>
-  <xacro:arg name="use_gazebo_camera" default="false"/>
-  <xacro:arg name="other_geometry_config_file"
+  <xacro:arg
+    name="robot_spec_config_file"
+    default="$(find xarm_description)/config/default_urdf_arguments/xarm6.yaml"
+  />
+  <xacro:property
+    name="robot_spec_config_file"
+    value="$(arg robot_spec_config_file)"
+  />
+  <xacro:property
+    name="robot_spec"
+    value="${xacro.load_yaml(robot_spec_config_file)}" />
+  <xacro:arg
+    name="end_effector_config_file"
+    default="$(find xarm_description)/config/default_urdf_arguments/end_effector.yaml"
+  />
+  <xacro:property
+    name="end_effector_config_file"
+    value="$(arg end_effector_config_file)"
+  />
+  <xacro:property
+    name="add_end_effector"
+    value="${xacro.load_yaml(end_effector_config_file)}"
+  />
+  <xacro:arg
+    name="other_geometry_config_file"
     default="$(find xarm_description)/config/default_urdf_arguments/other_geometry.yaml"
   />
-  <xacro:property name="other_geometry_config_file" value="$(arg other_geometry_config_file)" />
+  <xacro:property
+    name="other_geometry_config_file"
+    value="$(arg other_geometry_config_file)"
+  />
   <xacro:property name="other_geometry"
     value="${xacro.load_yaml(other_geometry_config_file)}"
   />
-  <xacro:arg name="baud_checkset" default="true"/>
-  <xacro:arg name="default_gripper_baud" default="2000000"/>
-  <xacro:arg name="attach_to" default="world"/>
-  <xacro:arg name="attach_xyz" default="0 0 0"/>
-  <xacro:arg name="attach_rpy" default="0 0 0"/>
-  <xacro:arg name="mesh_suffix" default="stl"/>
-  <xacro:arg name="kinematics_suffix" default=""/>
   <!-- load xarm device -->
   <xacro:include filename="$(find xarm_description)/urdf/xarm_device_macro.xacro" />
@@ -42,26 +52,26 @@
     ros2_control_plugin="$(arg ros2_control_plugin)"
     ros2_control_params="$(arg ros2_control_params)"
-    robot_ip="$(arg robot_ip)"
-    dof="$(arg dof)"
-    robot_type="$(arg robot_type)"
-    report_type="$(arg report_type)"
-    baud_checkset="$(arg baud_checkset)"
-    default_gripper_baud="$(arg default_gripper_baud)"
-    model1300="$(arg model1300)"
-    robot_sn="$(arg robot_sn)"
-    limited="$(arg limited)"
-    effort_control="$(arg effort_control)"
-    velocity_control="$(arg velocity_control)"
-    attach_to="$(arg attach_to)"
-    attach_xyz="$(arg attach_xyz)"
-    attach_rpy="$(arg attach_rpy)"
-    add_gripper="$(arg add_gripper)"
-    add_vacuum_gripper="$(arg add_vacuum_gripper)"
-    add_bio_gripper="$(arg add_bio_gripper)"
-    add_realsense_d435i="$(arg add_realsense_d435i)"
-    add_d435i_links="$(arg add_d435i_links)"
-    mesh_suffix="$(arg mesh_suffix)"
-    kinematics_suffix="$(arg kinematics_suffix)"
-    use_gazebo_camera="$(arg use_gazebo_camera)"
+    robot_ip="${robot_spec['robot_ip']}"
+    dof="${robot_spec['dof']}"
+    robot_type="${robot_spec['robot_type']}"
+    report_type="${robot_spec['report_type']}"
+    baud_checkset="${robot_spec['baud_checkset']}"
+    default_gripper_baud="${robot_spec['default_gripper_baud']}"
+    model1300="${robot_spec['model1300']}"
+    robot_sn="${robot_spec['robot_sn']}"
+    limited="${robot_spec['limited']}"
+    effort_control="${robot_spec['effort_control']}"
+    velocity_control="${robot_spec['velocity_control']}"
+    attach_to="${robot_spec['attach_to']}"
+    attach_xyz="${robot_spec['attach_xyz']}"
+    attach_rpy="${robot_spec['attach_rpy']}"
+    mesh_suffix="${robot_spec['mesh_suffix']}"
+    kinematics_suffix="${robot_spec['kinematics_suffix']}"
+    add_gripper="${add_end_effector['gripper']}"
+    add_vacuum_gripper="${add_end_effector['vacuum_gripper']}"
+    add_bio_gripper="${add_end_effector['bio_gripper']}"
+    add_realsense_d435i="${add_end_effector['realsense_d435i']}"
+    add_d435i_links="${add_end_effector['d435i_links']}"
+    use_gazebo_camera="false"
     add_other_geometry="${other_geometry['add']}"
     geometry_type="${other_geometry['type']}"

Commit message: TF tree now connected, but robot falls over

File: xarm_description/urdf/xarm_device.urdf.xacro (robot description, xacro)
@@ -1,4 +1,4 @@
 <?xml version='1.0' encoding='utf-8'?>
-<robot xmlns:xacro="http://ros.org/wiki/xacro" name="UF_ROBOT">
+<robot xmlns:xacro="http://ros.org/wiki/xacro" name="xarm_device">
   <!-- macro for having property with the same name/value as an argument -->
   <xacro:macro name="define_arg_property" params="prop_name default">
@@ -66,4 +66,5 @@
     attach_xyz="${robot_spec['attach_xyz']}"
     attach_rpy="${robot_spec['attach_rpy']}"
+    create_attach_link="${robot_spec['create_attach_link']}"
     mesh_suffix="${robot_spec['mesh_suffix']}"
     kinematics_suffix="${robot_spec['kinematics_suffix']}"

File: xarm_description/urdf/xarm_device_macro.xacro (robot description, xacro)
@@ -64,12 +64,14 @@
     <xacro:property name="new_model1300" value="${scope_parent_model1300}"/>
     <!-- add one world link if no 'attach_to' specified  -->
-    <xacro:if value="${attach_to == 'world' and create_attach_link}">
-      <link name="world" />
-    </xacro:if>
-    <joint name="${prefix}world_joint" type="fixed">
-      <parent link="${attach_to}" />
-      <child link="${prefix}link_base" />
-      <origin xyz="${attach_xyz}" rpy="${attach_rpy}" />
-    </joint>
+    <xacro:if value="${attach_to != ''}">
+      <xacro:if value="${create_attach_link}">
+        <link name="${attach_to}" />
+      </xacro:if>
+      <joint name="${prefix}world_joint" type="fixed">
+        <parent link="${attach_to}" />
+        <child link="${prefix}link_base" />
+        <origin xyz="${attach_xyz}" rpy="${attach_rpy}" />
+      </joint>
+    </xacro:if>
     <xacro:if value="${effort_control}">
       <xacro:property name="hard_interface" value="EffortJointInterface" />
@@ -284,4 +286,18 @@
     </xacro:if>
     <xacro:device_macro_end />
+    <gazebo>
+        <plugin filename="ignition-gazebo-pose-publisher-system" name="gz::sim::systems::PosePublisher">
+            <publish_link_pose>false</publish_link_pose>
+            <publish_visual_pose>false</publish_visual_pose>
+            <publish_collision_pose>false</publish_collision_pose>
+            <publish_sensor_pose>false</publish_sensor_pose>
+            <publish_model_pose>true</publish_model_pose>
+            <publish_nested_model_pose>true</publish_nested_model_pose>
+            <use_pose_vector_msg>true</use_pose_vector_msg>
+            <update_frequency>10</update_frequency>
+            <static_publisher>false</static_publisher>
+            <static_update_frequency>10</static_update_frequency>
+        </plugin>
+    </gazebo>
   </xacro:macro>
 </robot>
