Commit message: fix tag

File: xarm_description/urdf/xarm_device_macro.xacro (robot description, xacro)
@@ -270,5 +270,5 @@
     </xacro:if>
     <xacro:unless value="${ros2_control_params != ''}">
-      <xacro:property name="new_ros2_control_params" value="${find xarm_controller/config/${robot_name}_controllers.yaml}" />
+      <xacro:property name="new_ros2_control_params" value="$(find xarm_controller)/config/${robot_name}_controllers.yaml" />
     </xacro:unless>
     <!-- Detect whether to use ignition or classic -->

Commit message: robot doesn't fall down now, but sim is slow

File: xarm_description/urdf/xarm_device_macro.xacro (robot description, xacro)
@@ -74,4 +74,21 @@
       </joint>
     </xacro:if>
+    <link name="${prefix}make_kinematic">
+      <gazebo>
+        <kinematic>true</kinematic>
+      </gazebo>
+      <inertial>
+        <origin xyz="0.0 0.0 0.0" rpy="0 0 0" />
+        <mass value="100" />
+        <inertia
+          ixx="1.0" ixy="-3.5E-06" ixz="1.25E-05"
+          iyy="1.0" iyz="1.67E-06" izz="1.0" />
+      </inertial>
+    </link>
+    <joint name="${prefix}make_kinematic_joint" type="fixed">
+      <parent link="${prefix}link_base" />
+      <child link="${prefix}make_kinematic" />
+      <origin xyz="0 0 0" rpy="0 0 0"/>
+    </joint>
     <xacro:if value="${effort_control}">
       <xacro:property name="hard_interface" value="EffortJointInterface" />

File: xarm_moveit_config/srdf/xarm.srdf.xacro (robot description, xacro)
@@ -1,4 +1,4 @@
 <?xml version="1.0" encoding="UTF-8"?>
-<robot xmlns:xacro="http://wiki.ros.org/xacro" name="UF_ROBOT">
+<robot xmlns:xacro="http://wiki.ros.org/xacro" name="xarm_device">
   <!-- parameters -->
   <xacro:arg name="prefix" default="" />

File: xarm_moveit_config/srdf/xarm_macro.srdf.xacro (robot description, xacro)
@@ -1,4 +1,4 @@
 <?xml version="1.0" encoding="UTF-8"?>
-<robot xmlns:xacro="http://wiki.ros.org/xacro" name="xarm_srdf">
+<robot xmlns:xacro="http://wiki.ros.org/xacro" name="xarm_device">
   <xacro:macro name="xarm_macro_srdf" params="prefix:='' dof:=7 robot_type:='xarm'
     add_gripper:='false' add_vacuum_gripper:='false' add_bio_gripper:='false' add_other_geometry:='false' ">

Commit message: remove the 'heavy' link

File: xarm_description/urdf/xarm_device_macro.xacro (robot description, xacro)
@@ -74,21 +74,4 @@
       </joint>
     </xacro:if>
-    <link name="${prefix}make_kinematic">
-      <gazebo>
-        <kinematic>true</kinematic>
-      </gazebo>
-      <inertial>
-        <origin xyz="0.0 0.0 0.0" rpy="0 0 0" />
-        <mass value="100" />
-        <inertia
-          ixx="1.0" ixy="-3.5E-06" ixz="1.25E-05"
-          iyy="1.0" iyz="1.67E-06" izz="1.0" />
-      </inertial>
-    </link>
-    <joint name="${prefix}make_kinematic_joint" type="fixed">
-      <parent link="${prefix}link_base" />
-      <child link="${prefix}make_kinematic" />
-      <origin xyz="0 0 0" rpy="0 0 0"/>
-    </joint>
     <xacro:if value="${effort_control}">
       <xacro:property name="hard_interface" value="EffortJointInterface" />

Commit message: Fix TF tree (#10)
* TF tree now connected, but robot falls over

* robot doesn't fall down now, but sim is slow

* use keti_gz_utils create instead

* remove the 'heavy' link

---------

Co-authored-by: brian <brian@erl-brian>

File: xarm_description/urdf/xarm_device_macro.xacro (robot description, xacro)
@@ -64,12 +64,14 @@
     <xacro:property name="new_model1300" value="${scope_parent_model1300}"/>
     <!-- add one world link if no 'attach_to' specified  -->
-    <xacro:if value="${attach_to == 'world' and create_attach_link}">
-      <link name="world" />
-    </xacro:if>
-    <joint name="${prefix}world_joint" type="fixed">
-      <parent link="${attach_to}" />
-      <child link="${prefix}link_base" />
-      <origin xyz="${attach_xyz}" rpy="${attach_rpy}" />
-    </joint>
+    <xacro:if value="${attach_to != ''}">
+      <xacro:if value="${create_attach_link}">
+        <link name="${attach_to}" />
+      </xacro:if>
+      <joint name="${prefix}world_joint" type="fixed">
+        <parent link="${attach_to}" />
+        <child link="${prefix}link_base" />
+        <origin xyz="${attach_xyz}" rpy="${attach_rpy}" />
+      </joint>
+    </xacro:if>
     <xacro:if value="${effort_control}">
       <xacro:property name="hard_interface" value="EffortJointInterface" />
@@ -284,4 +286,18 @@
     </xacro:if>
     <xacro:device_macro_end />
+    <gazebo>
+        <plugin filename="ignition-gazebo-pose-publisher-system" name="gz::sim::systems::PosePublisher">
+            <publish_link_pose>false</publish_link_pose>
+            <publish_visual_pose>false</publish_visual_pose>
+            <publish_collision_pose>false</publish_collision_pose>
+            <publish_sensor_pose>false</publish_sensor_pose>
+            <publish_model_pose>true</publish_model_pose>
+            <publish_nested_model_pose>true</publish_nested_model_pose>
+            <use_pose_vector_msg>true</use_pose_vector_msg>
+            <update_frequency>10</update_frequency>
+            <static_publisher>false</static_publisher>
+            <static_update_frequency>10</static_update_frequency>
+        </plugin>
+    </gazebo>
   </xacro:macro>
 </robot>
