Commit message: Adding gripper

File: xarm_description/urdf/xarm6/xarm6.urdf.xacro (robot description, xacro)
@@ -99,5 +99,5 @@
       <parent link="${prefix}link1"/>
       <child link="${prefix}link2"/>
-      <!-- <origin xyz="0 0 0" rpy="-1.5708 0 0" /> -->
+      <origin xyz="0 0 0" rpy="-1.5708 -0.5 0" />
       <xacro:common_joint_origin joint_kinematic_params="${kinematics_params['joint2']}" />
       <axis xyz="0 0 1"/>
@@ -126,5 +126,5 @@
       <parent link="${prefix}link2"/>
       <child link="${prefix}link3"/>
-      <!-- <origin xyz="0.0535 -0.2845 0" rpy="0 0 0"/> -->
+      <origin xyz="0.0535 -0.2845 0" rpy="0 0 -0.5"/>
       <xacro:common_joint_origin joint_kinematic_params="${kinematics_params['joint3']}" />
       <axis xyz="0 0 1"/>
@@ -180,4 +180,5 @@
       <parent link="${prefix}link4"/>
       <child link="${prefix}link5"/>
+      <origin xyz="0.0 0.0 0.0" rpy="1.5708 -0.95 0.0"/>
       <xacro:common_joint_origin joint_kinematic_params="${kinematics_params['joint5']}" />
       <axis xyz="0 0 1"/>

Commit message: use different kinematics yaml between sim and real

File: xarm_description/urdf/xarm6/xarm6.urdf.xacro (robot description, xacro)
@@ -99,5 +99,5 @@
       <parent link="${prefix}link1"/>
       <child link="${prefix}link2"/>
-      <origin xyz="0 0 0" rpy="-1.5708 -0.5 0" />
+      <!-- <origin xyz="0 0 0" rpy="-1.5708 -0.5 0" /> -->
       <xacro:common_joint_origin joint_kinematic_params="${kinematics_params['joint2']}" />
       <axis xyz="0 0 1"/>
@@ -126,5 +126,5 @@
       <parent link="${prefix}link2"/>
       <child link="${prefix}link3"/>
-      <origin xyz="0.0535 -0.2845 0" rpy="0 0 -0.5"/>
+      <!-- <origin xyz="0.0535 -0.2845 0" rpy="0 0 -0.5"/> -->
       <xacro:common_joint_origin joint_kinematic_params="${kinematics_params['joint3']}" />
       <axis xyz="0 0 1"/>
@@ -180,5 +180,5 @@
       <parent link="${prefix}link4"/>
       <child link="${prefix}link5"/>
-      <origin xyz="0.0 0.0 0.0" rpy="1.5708 -0.95 0.0"/>
+      <!-- <origin xyz="0.0 0.0 0.0" rpy="1.5708 -0.95 0.0"/> -->
       <xacro:common_joint_origin joint_kinematic_params="${kinematics_params['joint5']}" />
       <axis xyz="0 0 1"/>

File: xarm_description/urdf/xarm_device.urdf.xacro (robot description, xacro)
@@ -10,4 +10,5 @@
   <xacro:arg name="ros2_control_plugin" default="uf_robot_hardware/UFRobotSystemHardware"/>
   <xacro:arg name="ros2_control_params" default=""/>
+  <xacro:arg name="kinematics_suffix" default=""/>
   <xacro:arg
     name="robot_spec_config_file"
@@ -68,5 +69,5 @@
     create_attach_link="${robot_spec['create_attach_link']}"
     mesh_suffix="${robot_spec['mesh_suffix']}"
-    kinematics_suffix="${robot_spec['kinematics_suffix']}"
+    kinematics_suffix="$(arg kinematics_suffix)"
     add_gripper="${add_end_effector['gripper']}"
     add_vacuum_gripper="${add_end_effector['vacuum_gripper']}"

Commit message: [Fixed Gripper]

File: xarm_description/urdf/xarm6/xarm6.urdf.xacro (robot description, xacro)
@@ -8,6 +8,8 @@
     joint5_lower_limit:=${-10*pi}  joint5_upper_limit:=${10*pi}
     joint6_lower_limit:=${-10*pi}  joint6_upper_limit:=${10*pi}
+    driver_joint:='0.85'
     model_num:=0
-    inertial_params_filename:='' kinematics_params_filename:='' "
+    inertial_params_filename:='' kinematics_params_filename:='' lock_gripper:='true'
+    "
     >
     <!-- define property -->
@@ -296,12 +298,22 @@
     </collision>
   </link>
-  <joint name="${prefix}drive_joint" type="revolute">
-    <origin rpy="0 0 0" xyz="0 0.035 0.059098"/>
-    <parent link="${prefix}xarm_gripper_base_link"/>
-    <child link="${prefix}left_outer_knuckle"/>
-    <axis xyz="1 0 0"/>
-    <limit effort="50" lower="0" upper="0.85" velocity="2"/>
-    <dynamics damping="1.0" friction="1.0"/>
-  </joint>
+  <xacro:if value="${lock_gripper}">
+    <joint name="${prefix}drive_joint" type="fixed">
+      <origin rpy="${driver_joint} 0 0" xyz="0 0.035 0.059098"/>
+      <parent link="${prefix}xarm_gripper_base_link"/>
+      <child  link="${prefix}left_outer_knuckle"/>
+    </joint>
+  </xacro:if>
+  <xacro:unless value="${lock_gripper}">
+    <joint name="${prefix}drive_joint" type="revolute">
+      <origin rpy="0 0 0" xyz="0 0.035 0.059098"/>
+      <parent link="${prefix}xarm_gripper_base_link"/>
+      <child  link="${prefix}left_outer_knuckle"/>
+      <axis xyz="1 0 0"/>
+      <limit effort="50" lower="0" upper="0.85" velocity="2"/>
+      <dynamics damping="1.0" friction="1.0"/>
+      <initial_position>0.0</initial_position>
+    </joint>
+  </xacro:unless>
   <link name="${prefix}left_finger">
     <inertial>
@@ -324,13 +336,22 @@
     </collision>
   </link>
-  <joint name="${prefix}left_finger_joint" type="revolute">
-    <origin rpy="0 0 0" xyz="0 0.035465 0.042039"/>
-    <parent link="${prefix}left_outer_knuckle"/>
-    <child link="${prefix}left_finger"/>
-    <axis xyz="-1 0 0"/>
-    <limit effort="50" lower="0" upper="0.85" velocity="2"/>
-    <mimic joint="${prefix}drive_joint" multiplier="1" offset="0"/>
-    <dynamics damping="1.0" friction="1.0"/>
-  </joint>
+  <xacro:if value="${lock_gripper}">
+    <joint name="${prefix}left_finger_joint" type="fixed">
+      <origin rpy="-${driver_joint} 0 0" xyz="0 0.035465 0.042039"/>
+      <parent link="${prefix}left_outer_knuckle"/>
+      <child link="${prefix}left_finger"/>
+    </joint>
+  </xacro:if>
+  <xacro:unless value="${lock_gripper}">
+    <joint name="${prefix}left_finger_joint" type="revolute">
+      <origin rpy="0 0 0" xyz="0 0.035465 0.042039"/>
+      <parent link="${prefix}left_outer_knuckle"/>
+      <child link="${prefix}left_finger"/>
+      <axis xyz="-1 0 0"/>
+      <limit effort="50" lower="0" upper="0.85" velocity="2"/>
+      <mimic joint="${prefix}drive_joint" multiplier="1" offset="0"/>
+      <dynamics damping="1.0" friction="1.0"/>
+    </joint>
+  </xacro:unless>
   <link name="${prefix}left_inner_knuckle">
     <inertial>
@@ -353,13 +374,22 @@
     </collision>
   </link>
-  <joint name="${prefix}left_inner_knuckle_joint" type="revolute">
-    <origin rpy="0 0 0" xyz="0 0.02 0.074098"/>
-    <parent link="${prefix}xarm_gripper_base_link"/>
-    <child link="${prefix}left_inner_knuckle"/>
-    <axis xyz="1 0 0"/>
-    <limit effort="50" lower="0" upper="0.85" velocity="2"/>
-    <mimic joint="${prefix}drive_joint" multiplier="1" offset="0"/>
-    <dynamics damping="1.0" friction="1.0"/>
-  </joint>
+  <xacro:if value="${lock_gripper}">
+    <joint name="${prefix}left_inner_knuckle_joint" type="fixed">
+      <origin rpy="${driver_joint} 0 0" xyz="0 0.02 0.074098"/>
+      <parent link="${prefix}xarm_gripper_base_link"/>
+      <child link="${prefix}left_inner_knuckle"/>
+    </joint>
+  </xacro:if>
+  <xacro:unless value="${lock_gripper}">
+    <joint name="${prefix}left_inner_knuckle_joint" type="revolute">
+      <origin rpy="0 0 0" xyz="0 0.02 0.074098"/>
+      <parent link="${prefix}xarm_gripper_base_link"/>
+      <child link="${prefix}left_inner_knuckle"/>
+      <axis xyz="1 0 0"/>
+      <limit effort="50" lower="0" upper="0.85" velocity="2"/>
+      <mimic joint="${prefix}drive_joint" multiplier="1" offset="0"/>
+      <dynamics damping="1.0" friction="1.0"/>
+    </joint>
+  </xacro:unless>
   <link name="${prefix}right_outer_knuckle">
     <inertial>
@@ -382,13 +412,22 @@
     </collision>
   </link>
-  <joint name="${prefix}right_outer_knuckle_joint" type="revolute">
-    <origin rpy="0 0 0" xyz="0 -0.035 0.059098"/>
-    <parent link="${prefix}xarm_gripper_base_link"/>
-    <child link="${prefix}right_outer_knuckle"/>
-    <axis xyz="-1 0 0"/>
-    <limit effort="50" lower="0" upper="0.85" velocity="2"/>
-    <mimic joint="${prefix}drive_joint" multiplier="1" offset="0"/>
-    <dynamics damping="1.0" friction="1.0"/>
-  </joint>
+  <xacro:if value="${lock_gripper}">
+    <joint name="${prefix}right_outer_knuckle_joint" type="fixed">
+      <origin rpy="-${driver_joint} 0 0" xyz="0 -0.035 0.059098"/>
+      <parent link="${prefix}xarm_gripper_base_link"/>
+      <child link="${prefix}right_outer_knuckle"/>
+    </joint>
+  </xacro:if>
+  <xacro:unless value="${lock_gripper}">
+    <joint name="${prefix}right_outer_knuckle_joint" type="revolute">
+      <origin rpy="0 0 0" xyz="0 -0.035 0.059098"/>
+      <parent link="${prefix}xarm_gripper_base_link"/>
+      <child link="${prefix}right_outer_knuckle"/>
+      <axis xyz="-1 0 0"/>
+      <limit effort="50" lower="0" upper="0.85" velocity="2"/>
+      <mimic joint="${prefix}drive_joint" multiplier="1" offset="0"/>
+      <dynamics damping="1.0" friction="1.0"/>
+    </joint>
+  </xacro:unless>
   <link name="${prefix}right_finger">
     <inertial>
@@ -411,13 +450,22 @@
     </collision>
   </link>
-  <joint name="${prefix}right_finger_joint" type="revolute">
-    <origin rpy="0 0 0" xyz="0 -0.035465 0.042039"/>
-    <parent link="${prefix}right_outer_knuckle"/>
-    <child link="${prefix}right_finger"/>
-    <axis xyz="1 0 0"/>
-    <limit effort="50" lower="0" upper="0.85" velocity="2"/>
-    <mimic joint="${prefix}drive_joint" multiplier="1" offset="0"/>
-    <dynamics damping="1.0" friction="1.0"/>
-  </joint>
+  <xacro:if value="${lock_gripper}">
+    <joint name="${prefix}right_finger_joint" type="fixed">
+      <origin rpy="${driver_joint} 0 0" xyz="0 -0.035465 0.042039"/>
+      <parent link="${prefix}right_outer_knuckle"/>
+      <child link="${prefix}right_finger"/>
+    </joint>
+  </xacro:if>
+  <xacro:unless value="${lock_gripper}">
+    <joint name="${prefix}right_finger_joint" type="revolute">
+      <origin rpy="0 0 0" xyz="0 -0.035465 0.042039"/>
+      <parent link="${prefix}right_outer_knuckle"/>
+      <child link="${prefix}right_finger"/>
+      <axis xyz="1 0 0"/>
+      <limit effort="50" lower="0" upper="0.85" velocity="2"/>
+      <mimic joint="${prefix}drive_joint" multiplier="1" offset="0"/>
+      <dynamics damping="1.0" friction="1.0"/>
+    </joint>
+  </xacro:unless>
   <link name="${prefix}right_inner_knuckle">
     <inertial>
@@ -440,15 +488,24 @@
     </collision>
   </link>
-  <joint name="${prefix}right_inner_knuckle_joint" type="revolute">
-    <origin rpy="0 0 0" xyz="0 -0.02 0.074098"/>
-    <parent link="${prefix}xarm_gripper_base_link"/>
-    <child link="${prefix}right_inner_knuckle"/>
-    <axis xyz="-1 0 0"/>
-    <limit effort="50" lower="0" upper="0.85" velocity="2"/>
-    <mimic joint="${prefix}drive_joint" multiplier="1" offset="0"/>
-    <dynamics damping="1.0" friction="1.0"/>
-  </joint>
+  <xacro:if value="${lock_gripper}">
+    <joint name="${prefix}right_inner_knuckle_joint" type="fixed">
+      <origin rpy="-${driver_joint} 0 0" xyz="0 -0.02 0.074098"/>
+      <parent link="${prefix}xarm_gripper_base_link"/>
+      <child link="${prefix}right_inner_knuckle"/>
+    </joint>
+  </xacro:if>
+  <xacro:unless value="${lock_gripper}">
+    <joint name="${prefix}right_inner_knuckle_joint" type="revolute">
+      <origin rpy="0 0 0" xyz="0 -0.02 0.074098"/>
+      <parent link="${prefix}xarm_gripper_base_link"/>
+      <child link="${prefix}right_inner_knuckle"/>
+      <axis xyz="-1 0 0"/>
+      <limit effort="50" lower="0" upper="0.85" velocity="2"/>
+      <mimic joint="${prefix}drive_joint" multiplier="1" offset="0"/>
+      <dynamics damping="1.0" friction="1.0"/>
+    </joint>
+  </xacro:unless>
   <!-- Gripper ee_tip - replaces the stick ee_tip when gripper is attached -->
-  <link name="${prefix}gripper_ee_tip">
+  <!-- <link name="${prefix}gripper_ee_tip">
   </link>
   <joint name="${prefix}gripper_ee_tip_joint" type="fixed">
@@ -457,5 +514,5 @@
     <child link="${prefix}gripper_ee_tip"/>
     <axis xyz="0 0 0"/>
-  </joint>
+  </joint> -->
   </xacro:macro>
 </robot>

Commit message: sanity check of orientation

File: xarm_description/urdf/xarm6/xarm6.urdf.xacro (robot description, xacro)
@@ -506,13 +506,13 @@
     </joint>
   </xacro:unless>
-  <!-- Gripper ee_tip - replaces the stick ee_tip when gripper is attached -->
-  <!-- <link name="${prefix}gripper_ee_tip">
+  <!-- Gripper ee_tip -->
+  <link name="${prefix}gripper_ee_tip">
   </link>
   <joint name="${prefix}gripper_ee_tip_joint" type="fixed">
-    <origin rpy="0 0 0" xyz="0 0 0.055"/>
-    <parent link="${prefix}right_finger"/>
+    <origin rpy="0 0 0" xyz="0 0 0.17"/>
+    <parent link="${prefix}xarm_gripper_base_link"/>
     <child link="${prefix}gripper_ee_tip"/>
     <axis xyz="0 0 0"/>
-  </joint> -->
+  </joint>
   </xacro:macro>
 </robot>

File: xarm_description/urdf/xarm6/xarm6_gripper.urdf.xacro (robot description, xacro)
@@ -8,6 +8,8 @@
     joint5_lower_limit:=${-10*pi}  joint5_upper_limit:=${10*pi}
     joint6_lower_limit:=${-10*pi}  joint6_upper_limit:=${10*pi}
+    driver_joint:='0.85'
     model_num:=0
-    inertial_params_filename:='' kinematics_params_filename:='' "
+    inertial_params_filename:='' kinematics_params_filename:='' lock_gripper:='true'
+    "
     >
     <!-- define property -->
@@ -296,12 +298,22 @@
     </collision>
   </link>
-  <joint name="${prefix}drive_joint" type="revolute">
-    <origin rpy="0 0 0" xyz="0 0.035 0.059098"/>
-    <parent link="${prefix}xarm_gripper_base_link"/>
-    <child link="${prefix}left_outer_knuckle"/>
-    <axis xyz="1 0 0"/>
-    <limit effort="50" lower="0" upper="0.85" velocity="2"/>
-    <dynamics damping="1.0" friction="1.0"/>
-  </joint>
+  <xacro:if value="${lock_gripper}">
+    <joint name="${prefix}drive_joint" type="fixed">
+      <origin rpy="${driver_joint} 0 0" xyz="0 0.035 0.059098"/>
+      <parent link="${prefix}xarm_gripper_base_link"/>
+      <child  link="${prefix}left_outer_knuckle"/>
+    </joint>
+  </xacro:if>
+  <xacro:unless value="${lock_gripper}">
+    <joint name="${prefix}drive_joint" type="revolute">
+      <origin rpy="0 0 0" xyz="0 0.035 0.059098"/>
+      <parent link="${prefix}xarm_gripper_base_link"/>
+      <child  link="${prefix}left_outer_knuckle"/>
+      <axis xyz="1 0 0"/>
+      <limit effort="50" lower="0" upper="0.85" velocity="2"/>
+      <dynamics damping="1.0" friction="1.0"/>
+      <initial_position>0.0</initial_position>
+    </joint>
+  </xacro:unless>
   <link name="${prefix}left_finger">
     <inertial>
@@ -324,13 +336,22 @@
     </collision>
   </link>
-  <joint name="${prefix}left_finger_joint" type="revolute">
-    <origin rpy="0 0 0" xyz="0 0.035465 0.042039"/>
-    <parent link="${prefix}left_outer_knuckle"/>
-    <child link="${prefix}left_finger"/>
-    <axis xyz="-1 0 0"/>
-    <limit effort="50" lower="0" upper="0.85" velocity="2"/>
-    <mimic joint="${prefix}drive_joint" multiplier="1" offset="0"/>
-    <dynamics damping="1.0" friction="1.0"/>
-  </joint>
+  <xacro:if value="${lock_gripper}">
+    <joint name="${prefix}left_finger_joint" type="fixed">
+      <origin rpy="-${driver_joint} 0 0" xyz="0 0.035465 0.042039"/>
+      <parent link="${prefix}left_outer_knuckle"/>
+      <child link="${prefix}left_finger"/>
+    </joint>
+  </xacro:if>
+  <xacro:unless value="${lock_gripper}">
+    <joint name="${prefix}left_finger_joint" type="revolute">
+      <origin rpy="0 0 0" xyz="0 0.035465 0.042039"/>
+      <parent link="${prefix}left_outer_knuckle"/>
+      <child link="${prefix}left_finger"/>
+      <axis xyz="-1 0 0"/>
+      <limit effort="50" lower="0" upper="0.85" velocity="2"/>
+      <mimic joint="${prefix}drive_joint" multiplier="1" offset="0"/>
+      <dynamics damping="1.0" friction="1.0"/>
+    </joint>
+  </xacro:unless>
   <link name="${prefix}left_inner_knuckle">
     <inertial>
@@ -353,13 +374,22 @@
     </collision>
   </link>
-  <joint name="${prefix}left_inner_knuckle_joint" type="revolute">
-    <origin rpy="0 0 0" xyz="0 0.02 0.074098"/>
-    <parent link="${prefix}xarm_gripper_base_link"/>
-    <child link="${prefix}left_inner_knuckle"/>
-    <axis xyz="1 0 0"/>
-    <limit effort="50" lower="0" upper="0.85" velocity="2"/>
-    <mimic joint="${prefix}drive_joint" multiplier="1" offset="0"/>
-    <dynamics damping="1.0" friction="1.0"/>
-  </joint>
+  <xacro:if value="${lock_gripper}">
+    <joint name="${prefix}left_inner_knuckle_joint" type="fixed">
+      <origin rpy="${driver_joint} 0 0" xyz="0 0.02 0.074098"/>
+      <parent link="${prefix}xarm_gripper_base_link"/>
+      <child link="${prefix}left_inner_knuckle"/>
+    </joint>
+  </xacro:if>
+  <xacro:unless value="${lock_gripper}">
+    <joint name="${prefix}left_inner_knuckle_joint" type="revolute">
+      <origin rpy="0 0 0" xyz="0 0.02 0.074098"/>
+      <parent link="${prefix}xarm_gripper_base_link"/>
+      <child link="${prefix}left_inner_knuckle"/>
+      <axis xyz="1 0 0"/>
+      <limit effort="50" lower="0" upper="0.85" velocity="2"/>
+      <mimic joint="${prefix}drive_joint" multiplier="1" offset="0"/>
+      <dynamics damping="1.0" friction="1.0"/>
+    </joint>
+  </xacro:unless>
   <link name="${prefix}right_outer_knuckle">
     <inertial>
@@ -382,13 +412,22 @@
     </collision>
   </link>
-  <joint name="${prefix}right_outer_knuckle_joint" type="revolute">
-    <origin rpy="0 0 0" xyz="0 -0.035 0.059098"/>
-    <parent link="${prefix}xarm_gripper_base_link"/>
-    <child link="${prefix}right_outer_knuckle"/>
-    <axis xyz="-1 0 0"/>
-    <limit effort="50" lower="0" upper="0.85" velocity="2"/>
-    <mimic joint="${prefix}drive_joint" multiplier="1" offset="0"/>
-    <dynamics damping="1.0" friction="1.0"/>
-  </joint>
+  <xacro:if value="${lock_gripper}">
+    <joint name="${prefix}right_outer_knuckle_joint" type="fixed">
+      <origin rpy="-${driver_joint} 0 0" xyz="0 -0.035 0.059098"/>
+      <parent link="${prefix}xarm_gripper_base_link"/>
+      <child link="${prefix}right_outer_knuckle"/>
+    </joint>
+  </xacro:if>
+  <xacro:unless value="${lock_gripper}">
+    <joint name="${prefix}right_outer_knuckle_joint" type="revolute">
+      <origin rpy="0 0 0" xyz="0 -0.035 0.059098"/>
+      <parent link="${prefix}xarm_gripper_base_link"/>
+      <child link="${prefix}right_outer_knuckle"/>
+      <axis xyz="-1 0 0"/>
+      <limit effort="50" lower="0" upper="0.85" velocity="2"/>
+      <mimic joint="${prefix}drive_joint" multiplier="1" offset="0"/>
+      <dynamics damping="1.0" friction="1.0"/>
+    </joint>
+  </xacro:unless>
   <link name="${prefix}right_finger">
     <inertial>
@@ -411,13 +450,22 @@
     </collision>
   </link>
-  <joint name="${prefix}right_finger_joint" type="revolute">
-    <origin rpy="0 0 0" xyz="0 -0.035465 0.042039"/>
-    <parent link="${prefix}right_outer_knuckle"/>
-    <child link="${prefix}right_finger"/>
-    <axis xyz="1 0 0"/>
-    <limit effort="50" lower="0" upper="0.85" velocity="2"/>
-    <mimic joint="${prefix}drive_joint" multiplier="1" offset="0"/>
-    <dynamics damping="1.0" friction="1.0"/>
-  </joint>
+  <xacro:if value="${lock_gripper}">
+    <joint name="${prefix}right_finger_joint" type="fixed">
+      <origin rpy="${driver_joint} 0 0" xyz="0 -0.035465 0.042039"/>
+      <parent link="${prefix}right_outer_knuckle"/>
+      <child link="${prefix}right_finger"/>
+    </joint>
+  </xacro:if>
+  <xacro:unless value="${lock_gripper}">
+    <joint name="${prefix}right_finger_joint" type="revolute">
+      <origin rpy="0 0 0" xyz="0 -0.035465 0.042039"/>
+      <parent link="${prefix}right_outer_knuckle"/>
+      <child link="${prefix}right_finger"/>
+      <axis xyz="1 0 0"/>
+      <limit effort="50" lower="0" upper="0.85" velocity="2"/>
+      <mimic joint="${prefix}drive_joint" multiplier="1" offset="0"/>
+      <dynamics damping="1.0" friction="1.0"/>
+    </joint>
+  </xacro:unless>
   <link name="${prefix}right_inner_knuckle">
     <inertial>
@@ -440,19 +488,28 @@
     </collision>
   </link>
-  <joint name="${prefix}right_inner_knuckle_joint" type="revolute">
-    <origin rpy="0 0 0" xyz="0 -0.02 0.074098"/>
+  <xacro:if value="${lock_gripper}">
+    <joint name="${prefix}right_inner_knuckle_joint" type="fixed">
+      <origin rpy="-${driver_joint} 0 0" xyz="0 -0.02 0.074098"/>
+      <parent link="${prefix}xarm_gripper_base_link"/>
+      <child link="${prefix}right_inner_knuckle"/>
+    </joint>
+  </xacro:if>
+  <xacro:unless value="${lock_gripper}">
+    <joint name="${prefix}right_inner_knuckle_joint" type="revolute">
+      <origin rpy="0 0 0" xyz="0 -0.02 0.074098"/>
+      <parent link="${prefix}xarm_gripper_base_link"/>
+      <child link="${prefix}right_inner_knuckle"/>
+      <axis xyz="-1 0 0"/>
+      <limit effort="50" lower="0" upper="0.85" velocity="2"/>
+      <mimic joint="${prefix}drive_joint" multiplier="1" offset="0"/>
+      <dynamics damping="1.0" friction="1.0"/>
+    </joint>
+  </xacro:unless>
+  <!-- Gripper ee_tip -->
+  <link name="${prefix}gripper_ee_tip">
+  </link>
+  <joint name="${prefix}gripper_ee_tip_joint" type="fixed">
+    <origin rpy="0 0 0" xyz="0 0 0.17"/>
     <parent link="${prefix}xarm_gripper_base_link"/>
-    <child link="${prefix}right_inner_knuckle"/>
-    <axis xyz="-1 0 0"/>
-    <limit effort="50" lower="0" upper="0.85" velocity="2"/>
-    <mimic joint="${prefix}drive_joint" multiplier="1" offset="0"/>
-    <dynamics damping="1.0" friction="1.0"/>
-  </joint>
-  <!-- Gripper ee_tip - replaces the stick ee_tip when gripper is attached -->
-  <link name="${prefix}gripper_ee_tip">
-  </link>
-  <joint name="${prefix}gripper_ee_tip_joint" type="fixed">
-    <origin rpy="0 0 0" xyz="0 0 0.055"/>
-    <parent link="${prefix}right_finger"/>
     <child link="${prefix}gripper_ee_tip"/>
     <axis xyz="0 0 0"/>
