Commit message: set up for sim

File: xarm_description/urdf/xarm6/xarm6_stick.urdf.xacro (robot description, xacro)
@@ -250,29 +250,23 @@
       <initial_position>0.0</initial_position>
     </joint>
+  <!-- sim set up -->
   <link name="${prefix}ee_stick">
-    <inertial>
-      <origin xyz="0 0 0.089" rpy="0 0 0"/>
-      <mass value="0.01"/>
-      <inertia ixx="0.0001" ixy="0" ixz="0" iyy="0.0001" iyz="0" izz="0.00001"/>
-    </inertial>
     <visual>
       <geometry>
-        <cylinder length="0.178" radius="0.005"/>
+        <cylinder length="0.33" radius="0.01"/>
       </geometry>
-      <origin rpy="0 0 0" xyz="0 0 0.089"/>
-      <material name="Purple">
-        <color rgba="0.5 0 0.5 1"/>
-      </material>
+      <origin rpy="0 0 0" xyz="0 0 0.18"/>
+      <material name="Purple"/>
     </visual>
     <collision>
       <geometry>
-        <cylinder length="0.178" radius="0.005"/>
+        <cylinder length="0.33" radius="0.01"/>
       </geometry>
-      <origin rpy="0 0 0" xyz="0 0 0.089"/>
+      <origin rpy="0 0 0" xyz="0 0 0.18"/>
     </collision>
   </link>
   <joint name="${prefix}joint_ee_stick" type="fixed">
     <origin rpy="0 0 0" xyz="0 0 -0.015"/>
-    <parent link="${prefix}link6"/>
+    <parent link="link6"/>
     <child link="${prefix}ee_stick"/>
     <axis xyz="0 0 0"/>
@@ -281,5 +275,5 @@
   </link>
   <joint name="${prefix}joint_ee_tip" type="fixed">
-    <origin rpy="0 0 0" xyz="0 0 0.178"/>
+    <origin rpy="0 0 0" xyz="0 0 0.337"/>
     <parent link="${prefix}ee_stick"/>
     <child link="${prefix}ee_tip"/>

Commit message: update stick with isaac

File: xarm_description/urdf/xarm6/xarm6_stick.urdf.xacro (robot description, xacro)
@@ -250,21 +250,20 @@
       <initial_position>0.0</initial_position>
     </joint>
-  <!-- sim set up -->
   <link name="${prefix}ee_stick">
     <visual>
       <geometry>
-        <cylinder length="0.33" radius="0.01"/>
+        <cylinder length="0.20" radius="0.01"/>
       </geometry>
-      <origin rpy="0 0 0" xyz="0 0 0.18"/>
+      <origin rpy="0 0 0" xyz="0 0 0.115"/>
       <material name="Purple"/>
     </visual>
     <collision>
       <geometry>
-        <cylinder length="0.33" radius="0.01"/>
+        <cylinder length="0.20" radius="0.01"/>
       </geometry>
-      <origin rpy="0 0 0" xyz="0 0 0.18"/>
+      <origin rpy="0 0 0" xyz="0 0 0.115"/>
     </collision>
   </link>
-  <joint name="${prefix}joint_ee_stick" type="fixed">
+  <joint name="${prefix}ee_stick_link6" type="fixed">
     <origin rpy="0 0 0" xyz="0 0 -0.015"/>
     <parent link="link6"/>
@@ -274,6 +273,6 @@
   <link name="${prefix}ee_tip">
   </link>
-  <joint name="${prefix}joint_ee_tip" type="fixed">
-    <origin rpy="0 0 0" xyz="0 0 0.337"/>
+  <joint name="${prefix}ee_tip_stick" type="fixed">
+    <origin rpy="0 0 0" xyz="0 0 0.215"/>
     <parent link="${prefix}ee_stick"/>
     <child link="${prefix}ee_tip"/>
