Commit message: add stick

File: xarm_description/urdf/xarm6/xarm6_robot_macro.xacro (robot description, xacro)
@@ -22,5 +22,5 @@
       <xacro:include filename="$(find xarm_description)/urdf/xarm6/xarm6.ros2_control.xacro" />
     </xacro:if>
-    <xacro:include filename="$(find xarm_description)/urdf/xarm6/xarm6.urdf.xacro" />
+    <xacro:include filename="$(find xarm_description)/urdf/xarm6/xarm6_stick.urdf.xacro" />
     <xacro:include filename="$(find xarm_description)/urdf/xarm6/xarm6.transmission.xacro" />
     <xacro:include filename="$(find xarm_description)/urdf/xarm6/xarm6.gazebo.xacro" />

File: xarm_description/urdf/xarm6/xarm6_stick.urdf.xacro (robot description, xacro)
@@ -252,5 +252,5 @@
   <link name="${prefix}ee_stick">
     <inertial>
-      <origin xyz="0 0 0.16" rpy="0 0 0"/>
+      <origin xyz="0 0 0.089" rpy="0 0 0"/>
       <mass value="0.01"/>
       <inertia ixx="0.0001" ixy="0" ixz="0" iyy="0.0001" iyz="0" izz="0.00001"/>
@@ -258,7 +258,7 @@
     <visual>
       <geometry>
-        <cylinder length="0.35" radius="0.01"/>
+        <cylinder length="0.178" radius="0.005"/>
       </geometry>
-      <origin rpy="0 0 0" xyz="0 0 0.16"/>
+      <origin rpy="0 0 0" xyz="0 0 0.089"/>
       <material name="Purple">
         <color rgba="0.5 0 0.5 1"/>
@@ -267,7 +267,7 @@
     <collision>
       <geometry>
-        <cylinder length="0.35" radius="0.01"/>
+        <cylinder length="0.178" radius="0.005"/>
       </geometry>
-      <origin rpy="0 0 0" xyz="0 0 0.16"/>
+      <origin rpy="0 0 0" xyz="0 0 0.089"/>
     </collision>
   </link>
@@ -281,5 +281,5 @@
   </link>
   <joint name="${prefix}joint_ee_tip" type="fixed">
-    <origin rpy="0 0 0" xyz="0 0 0.335"/>
+    <origin rpy="0 0 0" xyz="0 0 0.178"/>
     <parent link="${prefix}ee_stick"/>
     <child link="${prefix}ee_tip"/>

Commit message: [Collision Geometry] Adding wrist camera and collision step

File: xarm_description/urdf/xarm6/xarm6_robot_macro.xacro (robot description, xacro)
@@ -67,4 +67,11 @@
     <xacro:xarm6_transmission prefix="${prefix}" hard_interface="${hard_interface}" />
     <xacro:xarm6_gazebo prefix="${prefix}" />
+    <xacro:property name="M_PI" value="3.1415926535897931" />
+    <link name="wrist_camera_link" />
+    <joint name="wrist_camera_link_joint" type="fixed">
+      <parent link="${prefix}link_eef" />
+      <child link="wrist_camera_link" />
+      <origin xyz="0.06746 -0.0175 0.0237" rpy="${M_PI} ${-M_PI/2} 0" />
+    </joint>
   </xacro:macro>
 </robot>

File: xarm_description/urdf/xarm6/xarm6_stick.urdf.xacro (robot description, xacro)
@@ -250,33 +250,243 @@
       <initial_position>0.0</initial_position>
     </joint>
-  <link name="${prefix}ee_stick">
-    <visual>
-      <geometry>
-        <cylinder length="0.20" radius="0.01"/>
-      </geometry>
-      <origin rpy="0 0 0" xyz="0 0 0.115"/>
-      <material name="Purple"/>
-    </visual>
-    <collision>
-      <geometry>
-        <cylinder length="0.20" radius="0.01"/>
-      </geometry>
-      <origin rpy="0 0 0" xyz="0 0 0.115"/>
-    </collision>
-  </link>
-  <joint name="${prefix}ee_stick_link6" type="fixed">
-    <origin rpy="0 0 0" xyz="0 0 -0.015"/>
-    <parent link="link6"/>
-    <child link="${prefix}ee_stick"/>
-    <axis xyz="0 0 0"/>
-  </joint>
-  <link name="${prefix}ee_tip">
-  </link>
-  <joint name="${prefix}ee_tip_stick" type="fixed">
-    <origin rpy="0 0 0" xyz="0 0 0.215"/>
-    <parent link="${prefix}ee_stick"/>
-    <child link="${prefix}ee_tip"/>
-    <axis xyz="0 0 0"/>
-  </joint>
+	<link name="xarm6_ee_stick">
+		<visual>
+		<geometry>
+			<cylinder length="0.173" radius="0.005"/>
+		</geometry>
+		<origin rpy="0 0 0" xyz="0 0 0.0865"/>
+		<material name="Purple"/>
+		</visual>
+		<collision>
+			<geometry>
+				<sphere radius="0.005"></sphere>
+			</geometry>
+			<origin xyz="0.0 0.0 0.0" rpy="0 0 0"></origin>
+		</collision>
+		<collision>
+			<geometry>
+				<sphere radius="0.005"></sphere>
+			</geometry>
+			<origin xyz="0.0 0.0 0.005" rpy="0 0 0"></origin>
+		</collision>
+		<collision>
+			<geometry>
+				<sphere radius="0.005"></sphere>
+			</geometry>
+			<origin xyz="0.0 0.0 0.01" rpy="0 0 0"></origin>
+		</collision>
+		<collision>
+			<geometry>
+				<sphere radius="0.005"></sphere>
+			</geometry>
+			<origin xyz="0.0 0.0 0.015" rpy="0 0 0"></origin>
+		</collision>
+		<collision>
+			<geometry>
+				<sphere radius="0.005"></sphere>
+			</geometry>
+			<origin xyz="0.0 0.0 0.020" rpy="0 0 0"></origin>
+		</collision>
+		<collision>
+			<geometry>
+				<sphere radius="0.005"></sphere>
+			</geometry>
+			<origin xyz="0.0 0.0 0.025" rpy="0 0 0"></origin>
+		</collision>
+		<collision>
+			<geometry>
+				<sphere radius="0.005"></sphere>
+			</geometry>
+			<origin xyz="0.0 0.0 0.03" rpy="0 0 0"></origin>
+		</collision>
+		<collision>
+			<geometry>
+				<sphere radius="0.005"></sphere>
+			</geometry>
+			<origin xyz="0.0 0.0 0.035" rpy="0 0 0"></origin>
+		</collision>
+		<collision>
+			<geometry>
+				<sphere radius="0.005"></sphere>
+			</geometry>
+			<origin xyz="0.0 0.0 0.04" rpy="0 0 0"></origin>
+		</collision>
+		<collision>
+			<geometry>
+				<sphere radius="0.005"></sphere>
+			</geometry>
+			<origin xyz="0.0 0.0 0.045" rpy="0 0 0"></origin>
+		</collision>
+		<collision>
+			<geometry>
+				<sphere radius="0.005"></sphere>
+			</geometry>
+			<origin xyz="0.0 0.0 0.05" rpy="0 0 0"></origin>
+		</collision>
+		<collision>
+			<geometry>
+				<sphere radius="0.005"></sphere>
+			</geometry>
+			<origin xyz="0.0 0.0 0.055" rpy="0 0 0"></origin>
+		</collision>
+		<collision>
+			<geometry>
+				<sphere radius="0.005"></sphere>
+			</geometry>
+			<origin xyz="0.0 0.0 0.06" rpy="0 0 0"></origin>
+		</collision>
+		<collision>
+			<geometry>
+				<sphere radius="0.005"></sphere>
+			</geometry>
+			<origin xyz="0.0 0.0 0.065" rpy="0 0 0"></origin>
+		</collision>
+		<collision>
+			<geometry>
+				<sphere radius="0.005"></sphere>
+			</geometry>
+			<origin xyz="0.0 0.0 0.07" rpy="0 0 0"></origin>
+		</collision>
+		<collision>
+			<geometry>
+				<sphere radius="0.005"></sphere>
+			</geometry>
+			<origin xyz="0.0 0.0 0.075" rpy="0 0 0"></origin>
+		</collision>
+		<collision>
+			<geometry>
+				<sphere radius="0.005"></sphere>
+			</geometry>
+			<origin xyz="0.0 0.0 0.08" rpy="0 0 0"></origin>
+		</collision>
+		<collision>
+			<geometry>
+				<sphere radius="0.005"></sphere>
+			</geometry>
+			<origin xyz="0.0 0.0 0.09" rpy="0 0 0"></origin>
+		</collision>
+		<collision>
+			<geometry>
+				<sphere radius="0.005"></sphere>
+			</geometry>
+			<origin xyz="0.0 0.0 0.095" rpy="0 0 0"></origin>
+		</collision>
+		<collision>
+			<geometry>
+				<sphere radius="0.005"></sphere>
+			</geometry>
+			<origin xyz="0.0 0.0 0.1" rpy="0 0 0"></origin>
+		</collision>
+		<collision>
+			<geometry>
+				<sphere radius="0.005"></sphere>
+			</geometry>
+			<origin xyz="0.0 0.0 0.105" rpy="0 0 0"></origin>
+		</collision>
+		<collision>
+			<geometry>
+				<sphere radius="0.005"></sphere>
+			</geometry>
+			<origin xyz="0.0 0.0 0.11" rpy="0 0 0"></origin>
+		</collision>
+		<collision>
+			<geometry>
+				<sphere radius="0.005"></sphere>
+			</geometry>
+			<origin xyz="0.0 0.0 0.115" rpy="0 0 0"></origin>
+		</collision>
+		<collision>
+			<geometry>
+				<sphere radius="0.005"></sphere>
+			</geometry>
+			<origin xyz="0.0 0.0 0.120" rpy="0 0 0"></origin>
+		</collision>
+		<collision>
+			<geometry>
+				<sphere radius="0.005"></sphere>
+			</geometry>
+			<origin xyz="0.0 0.0 0.125" rpy="0 0 0"></origin>
+		</collision>
+		<collision>
+			<geometry>
+				<sphere radius="0.005"></sphere>
+			</geometry>
+			<origin xyz="0.0 0.0 0.13" rpy="0 0 0"></origin>
+		</collision>
+		<collision>
+			<geometry>
+				<sphere radius="0.005"></sphere>
+			</geometry>
+			<origin xyz="0.0 0.0 0.135" rpy="0 0 0"></origin>
+		</collision>
+		<collision>
+			<geometry>
+				<sphere radius="0.005"></sphere>
+			</geometry>
+			<origin xyz="0.0 0.0 0.14" rpy="0 0 0"></origin>
+		</collision>
+		<collision>
+			<geometry>
+				<sphere radius="0.005"></sphere>
+			</geometry>
+			<origin xyz="0.0 0.0 0.145" rpy="0 0 0"></origin>
+		</collision>
+		<collision>
+			<geometry>
+				<sphere radius="0.005"></sphere>
+			</geometry>
+			<origin xyz="0.0 0.0 0.15" rpy="0 0 0"></origin>
+		</collision>
+		<collision>
+			<geometry>
+				<sphere radius="0.005"></sphere>
+			</geometry>
+			<origin xyz="0.0 0.0 0.155" rpy="0 0 0"></origin>
+		</collision>
+		<collision>
+			<geometry>
+				<sphere radius="0.005"></sphere>
+			</geometry>
+			<origin xyz="0.0 0.0 0.16" rpy="0 0 0"></origin>
+		</collision>
+		<collision>
+			<geometry>
+				<sphere radius="0.005"></sphere>
+			</geometry>
+			<origin xyz="0.0 0.0 0.165" rpy="0 0 0"></origin>
+		</collision>
+		<collision>
+			<geometry>
+				<sphere radius="0.005"></sphere>
+			</geometry>
+			<origin xyz="0.0 0.0 0.17" rpy="0 0 0"></origin>
+		</collision>
+		<collision>
+			<geometry>
+				<sphere radius="0.005"></sphere>
+			</geometry>
+			<origin xyz="0.0 0.0 0.175" rpy="0 0 0"></origin>
+		</collision>
+	</link>
+	<joint name="xarm6_ee_stick_joint" type="fixed">
+		<origin rpy="0 0 0" xyz="0 0 -0.015"/>
+		<parent link="${prefix}link6"/>
+		<child link="xarm6_ee_stick"/>
+		<axis xyz="0 0 0"/>
+	</joint>
+	<link name="xarm6_ee_tip">
+		<collision>
+			<geometry>
+				<sphere radius="0.01"></sphere>
+			</geometry>
+			<origin xyz="0.0 0.0 0.0" rpy="0 0 0"></origin>
+		</collision>
+	</link>
+	<joint name="xarm6_ee_tip_joint" type="fixed">
+		<origin rpy="0 0 0" xyz="0 0 0.173"/>
+		<parent link="xarm6_ee_stick"/>
+		<child link="xarm6_ee_tip"/>
+		<axis xyz="0 0 0"/>
+	</joint>
   </xacro:macro>
 </robot>

Commit message: update wrist camera position

File: xarm_description/urdf/xarm6/xarm6_robot_macro.xacro (robot description, xacro)
@@ -72,5 +72,5 @@
       <parent link="${prefix}link_eef" />
       <child link="wrist_camera_link" />
-      <origin xyz="0.06746 -0.0175 0.0237" rpy="${M_PI} ${-M_PI/2} 0" />
+      <origin xyz="0.06746 -0.0575 0.0237" rpy="${M_PI} ${-M_PI/2} 0" />
     </joint>
   </xacro:macro>
