Commit message: feat: update xarm6 configuration for MPPI Isaac control - Add ros2_control params configuration - Update CMakeLists and URDF for xarm6 - Add xarm6_push launch file and table_world.sdf - Update env_publisher and table world - Remove obsolete scripts and world files

File: xarm_description/urdf/xarm6/xarm6.ros2_control.xacro (robot description, xacro)
@@ -12,4 +12,6 @@
     joint5_lower_limit:=${-10*pi}  joint5_upper_limit:=${10*pi}
     joint6_lower_limit:=${-10*pi}  joint6_upper_limit:=${10*pi}">
+    <!-- Define initial joint position -->
+    <xacro:property name="init_joint_pos" value="${[0.0, -0.78, -0.78, 0.0, 1.5708, 0.0]}" />
     <ros2_control name="${prefix}${ros2_control_plugin}" type="system">
       <hardware>
@@ -44,5 +46,7 @@
           <param name="max">3.14</param>
         </command_interface>
-        <state_interface name="position"/>
+        <state_interface name="position">
+          <param name="initial_value">${init_joint_pos[0]}</param>
+        </state_interface>
         <state_interface name="velocity"/>
         <!-- <state_interface name="effort"/> -->
@@ -57,5 +61,7 @@
           <param name="max">3.14</param>
         </command_interface>
-        <state_interface name="position"/>
+        <state_interface name="position">
+          <param name="initial_value">${init_joint_pos[1]}</param>
+        </state_interface>
         <state_interface name="velocity"/>
         <!-- <state_interface name="effort"/> -->
@@ -70,5 +76,7 @@
           <param name="max">3.14</param>
         </command_interface>
-        <state_interface name="position"/>
+        <state_interface name="position">
+          <param name="initial_value">${init_joint_pos[2]}</param>
+        </state_interface>
         <state_interface name="velocity"/>
         <!-- <state_interface name="effort"/> -->
@@ -83,5 +91,7 @@
           <param name="max">3.14</param>
         </command_interface>
-        <state_interface name="position"/>
+        <state_interface name="position">
+          <param name="initial_value">${init_joint_pos[3]}</param>
+        </state_interface>
         <state_interface name="velocity"/>
         <!-- <state_interface name="effort"/> -->
@@ -96,5 +106,7 @@
           <param name="max">3.14</param>
         </command_interface>
-        <state_interface name="position"/>
+        <state_interface name="position">
+          <param name="initial_value">${init_joint_pos[4]}</param>
+        </state_interface>
         <state_interface name="velocity"/>
         <!-- <state_interface name="effort"/> -->
@@ -109,5 +121,7 @@
           <param name="max">3.14</param>
         </command_interface>
-        <state_interface name="position"/>
+        <state_interface name="position">
+          <param name="initial_value">${init_joint_pos[5]}</param>
+        </state_interface>
         <state_interface name="velocity"/>
         <!-- <state_interface name="effort"/> -->

Commit message: [MPPI-Isaac] Integrated code into xarm_ros2 mppi branch.

File: xarm_description/urdf/xarm6/xarm6.ros2_control.xacro (robot description, xacro)
@@ -6,10 +6,12 @@
     hw_ns:='xarm' add_gripper:='false' add_bio_gripper:='false'
     robot_ip:='' report_type:='normal' baud_checkset:='true' default_gripper_baud:=2000000
-    joint1_lower_limit:=${-2.0*pi}  joint1_upper_limit:=${2.0*pi}
-    joint2_lower_limit:=${-2.059}  joint2_upper_limit:=${2.0944}
-    joint3_lower_limit:=${-3.927}  joint3_upper_limit:=${0.19198}
-    joint4_lower_limit:=${-2.0*pi}  joint4_upper_limit:=${2.0*pi}
-    joint5_lower_limit:=${-1.69297}  joint5_upper_limit:=${pi}
-    joint6_lower_limit:=${-2.0*pi}  joint6_upper_limit:=${2.0*pi}">
+    joint1_lower_limit:=${-10*pi}  joint1_upper_limit:=${10*pi}
+    joint2_lower_limit:=${-10*pi}  joint2_upper_limit:=${10*pi}
+    joint3_lower_limit:=${-10*pi}  joint3_upper_limit:=${10*pi}
+    joint4_lower_limit:=${-10*pi}  joint4_upper_limit:=${10*pi}
+    joint5_lower_limit:=${-10*pi}  joint5_upper_limit:=${10*pi}
+    joint6_lower_limit:=${-10*pi}  joint6_upper_limit:=${10*pi}">
+    <!-- Define initial joint position -->
+    <xacro:property name="init_joint_pos" value="${[0.0, -0.78, -0.78, 0.0, 1.5708, 0.0]}" />
     <ros2_control name="${prefix}${ros2_control_plugin}" type="system">
       <hardware>
@@ -44,9 +46,7 @@
           <param name="max">3.14</param>
         </command_interface>
-        <!-- <command_interface name="effort">
-          <param name="min">-3.14</param>
-          <param name="max">3.14</param>
-        </command_interface> -->
-        <state_interface name="position"/>
+        <state_interface name="position">
+          <param name="initial_value">${init_joint_pos[0]}</param>
+        </state_interface>
         <state_interface name="velocity"/>
         <!-- <state_interface name="effort"/> -->
@@ -61,9 +61,7 @@
           <param name="max">3.14</param>
         </command_interface>
-        <!-- <command_interface name="effort">
-          <param name="min">-3.14</param>
-          <param name="max">3.14</param>
-        </command_interface> -->
-        <state_interface name="position"/>
+        <state_interface name="position">
+          <param name="initial_value">${init_joint_pos[1]}</param>
+        </state_interface>
         <state_interface name="velocity"/>
         <!-- <state_interface name="effort"/> -->
@@ -78,9 +76,7 @@
           <param name="max">3.14</param>
         </command_interface>
-        <!-- <command_interface name="effort">
-          <param name="min">-3.14</param>
-          <param name="max">3.14</param>
-        </command_interface> -->
-        <state_interface name="position"/>
+        <state_interface name="position">
+          <param name="initial_value">${init_joint_pos[2]}</param>
+        </state_interface>
         <state_interface name="velocity"/>
         <!-- <state_interface name="effort"/> -->
@@ -95,9 +91,7 @@
           <param name="max">3.14</param>
         </command_interface>
-        <!-- <command_interface name="effort">
-          <param name="min">-3.14</param>
-          <param name="max">3.14</param>
-        </command_interface> -->
-        <state_interface name="position"/>
+        <state_interface name="position">
+          <param name="initial_value">${init_joint_pos[3]}</param>
+        </state_interface>
         <state_interface name="velocity"/>
         <!-- <state_interface name="effort"/> -->
@@ -112,9 +106,7 @@
           <param name="max">3.14</param>
         </command_interface>
-        <!-- <command_interface name="effort">
-          <param name="min">-3.14</param>
-          <param name="max">3.14</param>
-        </command_interface> -->
-        <state_interface name="position"/>
+        <state_interface name="position">
+          <param name="initial_value">${init_joint_pos[4]}</param>
+        </state_interface>
         <state_interface name="velocity"/>
         <!-- <state_interface name="effort"/> -->
@@ -129,11 +121,24 @@
           <param name="max">3.14</param>
         </command_interface>
-        <!-- <command_interface name="effort">
-          <param name="min">-3.14</param>
-          <param name="max">3.14</param>
-        </command_interface> -->
-        <state_interface name="position"/>
+        <state_interface name="position">
+          <param name="initial_value">${init_joint_pos[5]}</param>
+        </state_interface>
         <state_interface name="velocity"/>
         <!-- <state_interface name="effort"/> -->
+      </joint>
+      <!-- Gripper drive joint -->
+      <joint name="${prefix}drive_joint">
+        <command_interface name="position">
+          <param name="min">0</param>
+          <param name="max">0.85</param>
+        </command_interface>
+        <command_interface name="velocity">
+          <param name="min">-2.0</param>
+          <param name="max">2.0</param>
+        </command_interface>
+        <state_interface name="position">
+          <param name="initial_value">0.85</param>
+        </state_interface>
+        <state_interface name="velocity"/>
       </joint>
     </ros2_control>

File: xarm_description/urdf/xarm6/xarm6_gripper.urdf.xacro (robot description, xacro)
@@ -250,38 +250,210 @@
       <initial_position>0.0</initial_position>
     </joint>
-  <link name="${prefix}ee_stick">
-    <inertial>
-      <origin xyz="0 0 0.16" rpy="0 0 0"/>
-      <mass value="0.01"/>
-      <inertia ixx="0.0001" ixy="0" ixz="0" iyy="0.0001" iyz="0" izz="0.00001"/>
-    </inertial>
-    <visual>
-      <geometry>
-        <cylinder length="0.35" radius="0.01"/>
-      </geometry>
-      <origin rpy="0 0 0" xyz="0 0 0.16"/>
-      <material name="Purple">
-        <color rgba="0.5 0 0.5 1"/>
-      </material>
-    </visual>
-    <collision>
-      <geometry>
-        <cylinder length="0.35" radius="0.01"/>
-      </geometry>
-      <origin rpy="0 0 0" xyz="0 0 0.16"/>
-    </collision>
-  </link>
-  <joint name="${prefix}joint_ee_stick" type="fixed">
-    <origin rpy="0 0 0" xyz="0 0 -0.015"/>
+  <!-- Gripper components -->
+  <joint name="${prefix}gripper_fix" type="fixed">
     <parent link="${prefix}link6"/>
-    <child link="${prefix}ee_stick"/>
-    <axis xyz="0 0 0"/>
-  </joint>
-  <link name="${prefix}ee_tip">
-  </link>
-  <joint name="${prefix}joint_ee_tip" type="fixed">
-    <origin rpy="0 0 0" xyz="0 0 0.335"/>
-    <parent link="${prefix}ee_stick"/>
-    <child link="${prefix}ee_tip"/>
+    <child link="${prefix}xarm_gripper_base_link"/>
+    <origin rpy="0 0 0" xyz="0 0 0"/>
+  </joint>
+  <link name="${prefix}xarm_gripper_base_link">
+    <inertial>
+      <origin rpy="0 0 0" xyz="-0.00065489 -0.0018497 0.048028"/>
+      <mass value="0.54156"/>
+      <inertia ixx="0.00047106" ixy="3.9292E-07" ixz="2.6537E-06" iyy="0.00033072" iyz="-1.0975E-05" izz="0.00025642"/>
+    </inertial>
+    <visual>
+      <origin rpy="0 0 0" xyz="0 0 0"/>
+      <geometry>
+        <mesh filename="${mesh_path}/gripper/xarm/base_link.stl"/>
+      </geometry>
+      <material name="${prefix}White"/>
+    </visual>
+    <collision>
+      <origin rpy="0 0 0" xyz="0 0 0"/>
+      <geometry>
+        <mesh filename="${mesh_path}/gripper/xarm/base_link.stl"/>
+      </geometry>
+    </collision>
+  </link>
+  <link name="${prefix}left_outer_knuckle">
+    <inertial>
+      <origin rpy="0 0 0" xyz="2.9948E-14 0.021559 0.015181"/>
+      <mass value="0.033618"/>
+      <inertia ixx="1.9111E-05" ixy="-1.8803E-17" ixz="-1.1002E-17" iyy="6.6256E-06" iyz="-7.3008E-06" izz="1.3185E-05"/>
+    </inertial>
+    <visual>
+      <origin rpy="0 0 0" xyz="0 0 0"/>
+      <geometry>
+        <mesh filename="${mesh_path}/gripper/xarm/left_outer_knuckle.stl"/>
+      </geometry>
+      <material name="${prefix}Silver"/>
+    </visual>
+    <collision>
+      <origin rpy="0 0 0" xyz="0 0 0"/>
+      <geometry>
+        <mesh filename="${mesh_path}/gripper/xarm/left_outer_knuckle.stl"/>
+      </geometry>
+    </collision>
+  </link>
+  <joint name="${prefix}drive_joint" type="revolute">
+    <origin rpy="0 0 0" xyz="0 0.035 0.059098"/>
+    <parent link="${prefix}xarm_gripper_base_link"/>
+    <child link="${prefix}left_outer_knuckle"/>
+    <axis xyz="1 0 0"/>
+    <limit effort="50" lower="0" upper="0.85" velocity="2"/>
+    <dynamics damping="1.0" friction="1.0"/>
+  </joint>
+  <link name="${prefix}left_finger">
+    <inertial>
+      <origin rpy="0 0 0" xyz="-2.4536E-14 -0.016413 0.029258"/>
+      <mass value="0.048304"/>
+      <inertia ixx="1.7493E-05" ixy="-4.2156E-19" ixz="6.9164E-18" iyy="1.7225E-05" iyz="4.6433E-06" izz="5.1466E-06"/>
+    </inertial>
+    <visual>
+      <origin rpy="0 0 0" xyz="0 0 0"/>
+      <geometry>
+        <mesh filename="${mesh_path}/gripper/xarm/left_finger.stl"/>
+      </geometry>
+      <material name="${prefix}Silver"/>
+    </visual>
+    <collision>
+      <origin rpy="0 0 0" xyz="0 0 0"/>
+      <geometry>
+        <mesh filename="${mesh_path}/gripper/xarm/left_finger.stl"/>
+      </geometry>
+    </collision>
+  </link>
+  <joint name="${prefix}left_finger_joint" type="revolute">
+    <origin rpy="0 0 0" xyz="0 0.035465 0.042039"/>
+    <parent link="${prefix}left_outer_knuckle"/>
+    <child link="${prefix}left_finger"/>
+    <axis xyz="-1 0 0"/>
+    <limit effort="50" lower="0" upper="0.85" velocity="2"/>
+    <mimic joint="${prefix}drive_joint" multiplier="1" offset="0"/>
+    <dynamics damping="1.0" friction="1.0"/>
+  </joint>
+  <link name="${prefix}left_inner_knuckle">
+    <inertial>
+      <origin rpy="0 0 0" xyz="1.86600784687907E-06 0.0220467847633621 0.0261334672830885"/>
+      <mass value="0.0230125781256706"/>
+      <inertia ixx="6.09490024271906E-06" ixy="6.06651326160071E-11" ixz="7.19102670500635E-11" iyy="6.01955084375188E-06" iyz="-2.75316812991721E-06" izz="5.07862004479903E-06"/>
+    </inertial>
+    <visual>
+      <origin rpy="0 0 0" xyz="0 0 0"/>
+      <geometry>
+        <mesh filename="${mesh_path}/gripper/xarm/left_inner_knuckle.stl"/>
+      </geometry>
+      <material name="${prefix}Silver"/>
+    </visual>
+    <collision>
+      <origin rpy="0 0 0" xyz="0 0 0"/>
+      <geometry>
+        <mesh filename="${mesh_path}/gripper/xarm/left_inner_knuckle.stl"/>
+      </geometry>
+    </collision>
+  </link>
+  <joint name="${prefix}left_inner_knuckle_joint" type="revolute">
+    <origin rpy="0 0 0" xyz="0 0.02 0.074098"/>
+    <parent link="${prefix}xarm_gripper_base_link"/>
+    <child link="${prefix}left_inner_knuckle"/>
+    <axis xyz="1 0 0"/>
+    <limit effort="50" lower="0" upper="0.85" velocity="2"/>
+    <mimic joint="${prefix}drive_joint" multiplier="1" offset="0"/>
+    <dynamics damping="1.0" friction="1.0"/>
+  </joint>
+  <link name="${prefix}right_outer_knuckle">
+    <inertial>
+      <origin rpy="0 0 0" xyz="-3.1669E-14 -0.021559 0.015181"/>
+      <mass value="0.033618"/>
+      <inertia ixx="1.9111E-05" ixy="-1.8789E-17" ixz="1.0986E-17" iyy="6.6256E-06" iyz="7.3008E-06" izz="1.3185E-05"/>
+    </inertial>
+    <visual>
+      <origin rpy="0 0 0" xyz="0 0 0"/>
+      <geometry>
+        <mesh filename="${mesh_path}/gripper/xarm/right_outer_knuckle.stl"/>
+      </geometry>
+      <material name="${prefix}Silver"/>
+    </visual>
+    <collision>
+      <origin rpy="0 0 0" xyz="0 0 0"/>
+      <geometry>
+        <mesh filename="${mesh_path}/gripper/xarm/right_outer_knuckle.stl"/>
+      </geometry>
+    </collision>
+  </link>
+  <joint name="${prefix}right_outer_knuckle_joint" type="revolute">
+    <origin rpy="0 0 0" xyz="0 -0.035 0.059098"/>
+    <parent link="${prefix}xarm_gripper_base_link"/>
+    <child link="${prefix}right_outer_knuckle"/>
+    <axis xyz="-1 0 0"/>
+    <limit effort="50" lower="0" upper="0.85" velocity="2"/>
+    <mimic joint="${prefix}drive_joint" multiplier="1" offset="0"/>
+    <dynamics damping="1.0" friction="1.0"/>
+  </joint>
+  <link name="${prefix}right_finger">
+    <inertial>
+      <origin rpy="0 0 0" xyz="2.5618E-14 0.016413 0.029258"/>
+      <mass value="0.048304"/>
+      <inertia ixx="1.7493E-05" ixy="-5.0014E-19" ixz="-7.5079E-18" iyy="1.7225E-05" iyz="-4.6435E-06" izz="5.1466E-06"/>
+    </inertial>
+    <visual>
+      <origin rpy="0 0 0" xyz="0 0 0"/>
+      <geometry>
+        <mesh filename="${mesh_path}/gripper/xarm/right_finger.stl"/>
+      </geometry>
+      <material name="${prefix}Silver"/>
+    </visual>
+    <collision>
+      <origin rpy="0 0 0" xyz="0 0 0"/>
+      <geometry>
+        <mesh filename="${mesh_path}/gripper/xarm/right_finger.stl"/>
+      </geometry>
+    </collision>
+  </link>
+  <joint name="${prefix}right_finger_joint" type="revolute">
+    <origin rpy="0 0 0" xyz="0 -0.035465 0.042039"/>
+    <parent link="${prefix}right_outer_knuckle"/>
+    <child link="${prefix}right_finger"/>
+    <axis xyz="1 0 0"/>
+    <limit effort="50" lower="0" upper="0.85" velocity="2"/>
+    <mimic joint="${prefix}drive_joint" multiplier="1" offset="0"/>
+    <dynamics damping="1.0" friction="1.0"/>
+  </joint>
+  <link name="${prefix}right_inner_knuckle">
+    <inertial>
+      <origin rpy="0 0 0" xyz="1.866E-06 -0.022047 0.026133"/>
+      <mass value="0.023013"/>
+      <inertia ixx="6.0949E-06" ixy="-6.0665E-11" ixz="7.191E-11" iyy="6.0197E-06" iyz="2.7531E-06" izz="5.0784E-06"/>
+    </inertial>
+    <visual>
+      <origin rpy="0 0 0" xyz="0 0 0"/>
+      <geometry>
+        <mesh filename="${mesh_path}/gripper/xarm/right_inner_knuckle.stl"/>
+      </geometry>
+      <material name="${prefix}Silver"/>
+    </visual>
+    <collision>
+      <origin rpy="0 0 0" xyz="0 0 0"/>
+      <geometry>
+        <mesh filename="${mesh_path}/gripper/xarm/right_inner_knuckle.stl"/>
+      </geometry>
+    </collision>
+  </link>
+  <joint name="${prefix}right_inner_knuckle_joint" type="revolute">
+    <origin rpy="0 0 0" xyz="0 -0.02 0.074098"/>
+    <parent link="${prefix}xarm_gripper_base_link"/>
+    <child link="${prefix}right_inner_knuckle"/>
+    <axis xyz="-1 0 0"/>
+    <limit effort="50" lower="0" upper="0.85" velocity="2"/>
+    <mimic joint="${prefix}drive_joint" multiplier="1" offset="0"/>
+    <dynamics damping="1.0" friction="1.0"/>
+  </joint>
+  <!-- Gripper ee_tip - replaces the stick ee_tip when gripper is attached -->
+  <link name="${prefix}gripper_ee_tip">
+  </link>
+  <joint name="${prefix}gripper_ee_tip_joint" type="fixed">
+    <origin rpy="0 0 0" xyz="0 0 0.055"/>
+    <parent link="${prefix}right_finger"/>
+    <child link="${prefix}gripper_ee_tip"/>
     <axis xyz="0 0 0"/>
   </joint>

File: xarm_description/urdf/xarm_device.urdf.xacro (robot description, xacro)
@@ -10,5 +10,4 @@
   <xacro:arg name="ros2_control_plugin" default="uf_robot_hardware/UFRobotSystemHardware"/>
   <xacro:arg name="ros2_control_params" default=""/>
-  <xacro:arg name="kinematics_suffix" default=""/>
   <xacro:arg
     name="robot_spec_config_file"
@@ -59,5 +58,5 @@
     baud_checkset="${robot_spec['baud_checkset']}"
     default_gripper_baud="${robot_spec['default_gripper_baud']}"
-    model1300="${robot_spec['model1300']}"
+    model_num="${robot_spec['model_num']}"
     robot_sn="${robot_spec['robot_sn']}"
     limited="${robot_spec['limited']}"
@@ -69,5 +68,5 @@
     create_attach_link="${robot_spec['create_attach_link']}"
     mesh_suffix="${robot_spec['mesh_suffix']}"
-    kinematics_suffix="$(arg kinematics_suffix)"
+    kinematics_suffix="${robot_spec['kinematics_suffix']}"
     add_gripper="${add_end_effector['gripper']}"
     add_vacuum_gripper="${add_end_effector['vacuum_gripper']}"
