Commit message: Cleanup with latest -- using OI-MPPI
* Robot position

* _robot_joint_state.launch.py fixed

* moveit

* fix control launch

* propagate changes to gazebo

* Incorporating moveit in xarm6

* Moveit in besides_table world

* Incorporating moveit

* trying to revert namespacing

* works without namespace

* make single robot planning work

* Added camera and ros_gz_bridge node

* minor

* minor

* correct camera orientation

* Adding gripper

* minor

* octomap

* Fix TF tree (#10)

* TF tree now connected, but robot falls over

* robot doesn't fall down now, but sim is slow

* use keti_gz_utils create instead

* remove the 'heavy' link

---------

Co-authored-by: brian <brian@erl-brian>

* world_table.sdf changed

* Added [200~# Software License Agreement (BSD License)

* use a simple timer for the moment

* minor

* updated real robot_ip

* Gazebo velocity controller

* Velocity controller

* Controller specifing robot description

* use different kinematics yaml between sim and real

* Offset handling

* add user/xarm6_kinematics_sim.yaml

* minor

* [MPPI-Isaac] Integrated code into xarm_ros2 mppi branch.

* [Orient test] Match the limitation of joint velocity

* [Velocity Controller] Integrated

* [Gripper] Working on gripper

* [Fixed Gripper]

* Controller

* minor

* sanity check of orientation

* [Rviz] Finished MPPI visualization.

* Lab setup issue

* [Dev-mode] Joint state publishing frequency is 100 Hz

* add stick

* set up for sim

* update stick with isaac

* [Collision Geometry] Adding wrist camera and collision step

* wrist camera version

* update wrist camera position (#13)

Co-authored-by: Dwait Bhatt <dhbhatt@ucsd.edu>

---------

Co-authored-by: NikolaRaicevic <nikolar047@gmail.com>
Co-authored-by: Brian Lee <brian@UTS040524>
Co-authored-by: brian <brian@erl-brian>
Co-authored-by: Niyas-A <niyasttshr33@gmail.com>
Co-authored-by: Dwait Bhatt <dhbhatt@ucsd.edu>
Co-authored-by: NikolaRaicevic2001 <nmarinosraitsevits@ucsd.edu>
Co-authored-by: ticotico410 <ycb04106438which pip.com>

File: xarm_description/urdf/xarm6/xarm6.ros2_control.xacro (robot description, xacro)
@@ -6,10 +6,12 @@
     hw_ns:='xarm' add_gripper:='false' add_bio_gripper:='false'
     robot_ip:='' report_type:='normal' baud_checkset:='true' default_gripper_baud:=2000000
-    joint1_lower_limit:=${-2.0*pi}  joint1_upper_limit:=${2.0*pi}
-    joint2_lower_limit:=${-2.059}  joint2_upper_limit:=${2.0944}
-    joint3_lower_limit:=${-3.927}  joint3_upper_limit:=${0.19198}
-    joint4_lower_limit:=${-2.0*pi}  joint4_upper_limit:=${2.0*pi}
-    joint5_lower_limit:=${-1.69297}  joint5_upper_limit:=${pi}
-    joint6_lower_limit:=${-2.0*pi}  joint6_upper_limit:=${2.0*pi}">
+    joint1_lower_limit:=${-10*pi}  joint1_upper_limit:=${10*pi}
+    joint2_lower_limit:=${-10*pi}  joint2_upper_limit:=${10*pi}
+    joint3_lower_limit:=${-10*pi}  joint3_upper_limit:=${10*pi}
+    joint4_lower_limit:=${-10*pi}  joint4_upper_limit:=${10*pi}
+    joint5_lower_limit:=${-10*pi}  joint5_upper_limit:=${10*pi}
+    joint6_lower_limit:=${-10*pi}  joint6_upper_limit:=${10*pi}">
+    <!-- Define initial joint position -->
+    <xacro:property name="init_joint_pos" value="${[0.0, -0.78, -0.78, 0.0, 1.5708, 0.0]}" />
     <ros2_control name="${prefix}${ros2_control_plugin}" type="system">
       <hardware>
@@ -41,8 +43,10 @@
         </command_interface>
         <command_interface name="velocity">
-          <param name="min">-3.14</param>
-          <param name="max">3.14</param>
+          <param name="min">-0.2</param>
+          <param name="max">0.2</param>
         </command_interface>
-        <state_interface name="position"/>
+        <state_interface name="position">
+          <param name="initial_value">${init_joint_pos[0]}</param>
+        </state_interface>
         <state_interface name="velocity"/>
         <!-- <state_interface name="effort"/> -->
@@ -54,8 +58,10 @@
         </command_interface>
         <command_interface name="velocity">
-          <param name="min">-3.14</param>
-          <param name="max">3.14</param>
+          <param name="min">-0.2</param>
+          <param name="max">0.2</param>
         </command_interface>
-        <state_interface name="position"/>
+        <state_interface name="position">
+          <param name="initial_value">${init_joint_pos[1]}</param>
+        </state_interface>
         <state_interface name="velocity"/>
         <!-- <state_interface name="effort"/> -->
@@ -67,8 +73,10 @@
         </command_interface>
         <command_interface name="velocity">
-          <param name="min">-3.14</param>
-          <param name="max">3.14</param>
+          <param name="min">-0.2</param>
+          <param name="max">0.2</param>
         </command_interface>
-        <state_interface name="position"/>
+        <state_interface name="position">
+          <param name="initial_value">${init_joint_pos[2]}</param>
+        </state_interface>
         <state_interface name="velocity"/>
         <!-- <state_interface name="effort"/> -->
@@ -80,8 +88,10 @@
         </command_interface>
         <command_interface name="velocity">
-          <param name="min">-3.14</param>
-          <param name="max">3.14</param>
+          <param name="min">-0.2</param>
+          <param name="max">0.2</param>
         </command_interface>
-        <state_interface name="position"/>
+        <state_interface name="position">
+          <param name="initial_value">${init_joint_pos[3]}</param>
+        </state_interface>
         <state_interface name="velocity"/>
         <!-- <state_interface name="effort"/> -->
@@ -93,8 +103,10 @@
         </command_interface>
         <command_interface name="velocity">
-          <param name="min">-3.14</param>
-          <param name="max">3.14</param>
+          <param name="min">-0.2</param>
+          <param name="max">0.2</param>
         </command_interface>
-        <state_interface name="position"/>
+        <state_interface name="position">
+          <param name="initial_value">${init_joint_pos[4]}</param>
+        </state_interface>
         <state_interface name="velocity"/>
         <!-- <state_interface name="effort"/> -->
@@ -106,10 +118,27 @@
         </command_interface>
         <command_interface name="velocity">
-          <param name="min">-3.14</param>
-          <param name="max">3.14</param>
+          <param name="min">-0.2</param>
+          <param name="max">0.2</param>
         </command_interface>
-        <state_interface name="position"/>
+        <state_interface name="position">
+          <param name="initial_value">${init_joint_pos[5]}</param>
+        </state_interface>
         <state_interface name="velocity"/>
         <!-- <state_interface name="effort"/> -->
+      </joint>
+      <!-- Gripper drive joint -->
+      <joint name="${prefix}drive_joint">
+        <command_interface name="position">
+          <param name="min">0</param>
+          <param name="max">0.85</param>
+        </command_interface>
+        <command_interface name="velocity">
+          <param name="min">-2.0</param>
+          <param name="max">2.0</param>
+        </command_interface>
+        <state_interface name="position">
+          <param name="initial_value">0.85</param>
+        </state_interface>
+        <state_interface name="velocity"/>
       </joint>
     </ros2_control>
