Commit message: Cleanup with latest -- using OI-MPPI
* Robot position

* _robot_joint_state.launch.py fixed

* moveit

* fix control launch

* propagate changes to gazebo

* Incorporating moveit in xarm6

* Moveit in besides_table world

* Incorporating moveit

* trying to revert namespacing

* works without namespace

* make single robot planning work

* Added camera and ros_gz_bridge node

* minor

* minor

* correct camera orientation

* Adding gripper

* minor

* octomap

* Fix TF tree (#10)

* TF tree now connected, but robot falls over

* robot doesn't fall down now, but sim is slow

* use keti_gz_utils create instead

* remove the 'heavy' link

---------

Co-authored-by: brian <brian@erl-brian>

* world_table.sdf changed

* Added [200~# Software License Agreement (BSD License)

* use a simple timer for the moment

* minor

* updated real robot_ip

* Gazebo velocity controller

* Velocity controller

* Controller specifing robot description

* use different kinematics yaml between sim and real

* Offset handling

* add user/xarm6_kinematics_sim.yaml

* minor

* [MPPI-Isaac] Integrated code into xarm_ros2 mppi branch.

* [Orient test] Match the limitation of joint velocity

* [Velocity Controller] Integrated

* [Gripper] Working on gripper

* [Fixed Gripper]

* Controller

* minor

* sanity check of orientation

* [Rviz] Finished MPPI visualization.

* Lab setup issue

* [Dev-mode] Joint state publishing frequency is 100 Hz

* add stick

* set up for sim

* update stick with isaac

* [Collision Geometry] Adding wrist camera and collision step

* wrist camera version

* update wrist camera position (#13)

Co-authored-by: Dwait Bhatt <dhbhatt@ucsd.edu>

---------

Co-authored-by: NikolaRaicevic <nikolar047@gmail.com>
Co-authored-by: Brian Lee <brian@UTS040524>
Co-authored-by: brian <brian@erl-brian>
Co-authored-by: Niyas-A <niyasttshr33@gmail.com>
Co-authored-by: Dwait Bhatt <dhbhatt@ucsd.edu>
Co-authored-by: NikolaRaicevic2001 <nmarinosraitsevits@ucsd.edu>
Co-authored-by: ticotico410 <ycb04106438which pip.com>

File: xarm_description/urdf/xarm6/xarm6.urdf.xacro (robot description, xacro)
@@ -2,21 +2,37 @@
 <robot xmlns:xacro="http://ros.org/wiki/xacro">
   <xacro:macro name="xarm6_urdf" params="prefix
-    joint1_lower_limit:=${-2.0*pi}  joint1_upper_limit:=${2.0*pi}
-    joint2_lower_limit:=${-2.059}  joint2_upper_limit:=${2.0944}
-    joint3_lower_limit:=${-3.927}  joint3_upper_limit:=${0.19198}
-    joint4_lower_limit:=${-2.0*pi}  joint4_upper_limit:=${2.0*pi}
-    joint5_lower_limit:=${-1.69297}  joint5_upper_limit:=${pi}
-    joint6_lower_limit:=${-2.0*pi}  joint6_upper_limit:=${2.0*pi}
-    model1300:=false
-    inertial_params_filename:='' kinematics_params_filename:='' "
+    joint1_lower_limit:=${-10.0*pi}  joint1_upper_limit:=${10.0*pi}
+    joint2_lower_limit:=${-10*pi}  joint2_upper_limit:=${10*pi}
+    joint3_lower_limit:=${-10*pi}  joint3_upper_limit:=${10*pi}
+    joint4_lower_limit:=${-10*pi}  joint4_upper_limit:=${10*pi}
+    joint5_lower_limit:=${-10*pi}  joint5_upper_limit:=${10*pi}
+    joint6_lower_limit:=${-10*pi}  joint6_upper_limit:=${10*pi}
+    driver_joint:='0.85'
+    model_num:=0
+    inertial_params_filename:='' kinematics_params_filename:='' lock_gripper:='true'
+    "
     >
     <!-- define property -->
-    <xacro:if value="${model1300}">
-      <xacro:property name="end_tool_visual_filename" value="end_tool/visual/end_tool_1300"/>
-      <xacro:property name="end_tool_collision_filename" value="end_tool/collision/end_tool_1300"/>
+    <xacro:if value="${model_num >= 1305 and model_num != 1380}">
+      <xacro:property name="visual_dir" value="xarm6_1305/visual"/>
+      <xacro:property name="collision_dir" value="xarm6_1305/collision"/>
+      <xacro:property name="add_mesh_suffix" value="false"/>
+      <xacro:property name="collison_mesh_suffix" value="obj"/>
+      <xacro:property name="link6_visual" value="xarm6_1305/visual/link6"/>
+      <xacro:property name="link6_collision" value="xarm6_1305/collision/link6"/>
     </xacro:if>
-    <xacro:unless value="${model1300}">
-      <xacro:property name="end_tool_visual_filename" value="xarm6/visual/link6"/>
-      <xacro:property name="end_tool_collision_filename" value="end_tool/collision/end_tool"/>
+    <xacro:unless value="${model_num >= 1305 and model_num != 1380}">
+      <xacro:property name="visual_dir" value="xarm6/visual"/>
+      <xacro:property name="collision_dir" value="xarm6/visual"/>
+      <xacro:property name="add_mesh_suffix" value="true"/>
+      <xacro:property name="collison_mesh_suffix" value="stl"/>
+      <xacro:if value="${model_num >= 1300}">
+        <xacro:property name="link6_visual" value="end_tool/visual/end_tool_1300"/>
+        <xacro:property name="link6_collision" value="end_tool/collision/end_tool_1300"/>
+      </xacro:if>
+      <xacro:unless value="${model_num >= 1300}">
+        <xacro:property name="link6_visual" value="xarm6/visual/link6"/>
+        <xacro:property name="link6_collision" value="end_tool/collision/end_tool"/>
+      </xacro:unless>
     </xacro:unless>
     <!-- load params and define property -->
@@ -46,10 +62,12 @@
       </inertial>
       <xacro:common_link_visual
-        mesh_filename="xarm6/visual/link_base"
+        mesh_filename="${visual_dir}/link_base"
         origin_xyz="0 0 0"
         origin_rpy="0 0 0"
         material_name="${prefix}White" />
       <xacro:common_link_collision
-        mesh_filename="xarm6/visual/link_base"
+        mesh_filename="${collision_dir}/link_base"
+        add_mesh_suffix="${add_mesh_suffix}"
+        other_mesh_suffix="${collison_mesh_suffix}"
         origin_xyz="0 0 0"
         origin_rpy="0 0 0" />
@@ -60,10 +78,12 @@
         origin_rpy="0 0 0"/>
       <xacro:common_link_visual
-        mesh_filename="xarm6/visual/link1"
+        mesh_filename="${visual_dir}/link1"
         origin_xyz="0 0 0"
         origin_rpy="0 0 0"
         material_name="${prefix}White" />
       <xacro:common_link_collision
-        mesh_filename="xarm6/visual/link1"
+        mesh_filename="${collision_dir}/link1"
+        add_mesh_suffix="${add_mesh_suffix}"
+        other_mesh_suffix="${collison_mesh_suffix}"
         origin_xyz="0 0 0"
         origin_rpy="0 0 0" />
@@ -81,4 +101,5 @@
         velocity="3.14"/>
       <dynamics damping="1.0" friction="1.0"/>
+      <initial_position>0.0</initial_position>
     </joint>
     <link name="${prefix}link2">
@@ -87,11 +108,13 @@
         origin_rpy="0 0 0"/>
       <xacro:common_link_visual
-        mesh_filename="xarm6/visual/link2"
-        origin_xyz="0 0 ${-kinematics_params['joint2']['y']}"
+        mesh_filename="${visual_dir}/link2"
+        origin_xyz="0 0 0"
         origin_rpy="0 0 0"
         material_name="${prefix}White" />
       <xacro:common_link_collision
-        mesh_filename="xarm6/visual/link2"
-        origin_xyz="0 0 ${-kinematics_params['joint2']['y']}"
+        mesh_filename="${collision_dir}/link2"
+        add_mesh_suffix="${add_mesh_suffix}"
+        other_mesh_suffix="${collison_mesh_suffix}"
+        origin_xyz="0 0 0"
         origin_rpy="0 0 0" />
     </link>
@@ -108,4 +131,5 @@
         velocity="3.14"/>
       <dynamics damping="1.0" friction="1.0"/>
+      <initial_position>-0.78</initial_position>
     </joint>
     <link name="${prefix}link3">
@@ -114,10 +138,12 @@
         origin_rpy="0 0 0"/>
       <xacro:common_link_visual
-        mesh_filename="xarm6/visual/link3"
+        mesh_filename="${visual_dir}/link3"
         origin_xyz="0 0 0"
         origin_rpy="0 0 0"
         material_name="${prefix}White" />
       <xacro:common_link_collision
-        mesh_filename="xarm6/visual/link3"
+        mesh_filename="${collision_dir}/link3"
+        add_mesh_suffix="${add_mesh_suffix}"
+        other_mesh_suffix="${collison_mesh_suffix}"
         origin_xyz="0 0 0"
         origin_rpy="0 0 0" />
@@ -135,4 +161,5 @@
         velocity="3.14"/>
       <dynamics damping="1.0" friction="1.0"/>
+      <initial_position>-0.78</initial_position>
     </joint>
     <link name="${prefix}link4">
@@ -141,10 +168,12 @@
         origin_rpy="0 0 0"/>
       <xacro:common_link_visual
-        mesh_filename="xarm6/visual/link4"
+        mesh_filename="${visual_dir}/link4"
         origin_xyz="0 0 0"
         origin_rpy="0 0 0"
         material_name="${prefix}White" />
       <xacro:common_link_collision
-        mesh_filename="xarm6/visual/link4"
+        mesh_filename="${collision_dir}/link4"
+        add_mesh_suffix="${add_mesh_suffix}"
+        other_mesh_suffix="${collison_mesh_suffix}"
         origin_xyz="0 0 0"
         origin_rpy="0 0 0" />
@@ -162,4 +191,5 @@
         velocity="3.14"/>
       <dynamics damping="1.0" friction="1.0"/>
+      <initial_position>0.0</initial_position>
     </joint>
     <link name="${prefix}link5">
@@ -168,10 +198,12 @@
         origin_rpy="0 0 0"/>
       <xacro:common_link_visual
-        mesh_filename="xarm6/visual/link5"
+        mesh_filename="${visual_dir}/link5"
         origin_xyz="0 0 0"
         origin_rpy="0 0 0"
         material_name="${prefix}White" />
       <xacro:common_link_collision
-        mesh_filename="xarm6/visual/link5"
+        mesh_filename="${collision_dir}/link5"
+        add_mesh_suffix="${add_mesh_suffix}"
+        other_mesh_suffix="${collison_mesh_suffix}"
         origin_xyz="0 0 0"
         origin_rpy="0 0 0" />
@@ -188,4 +220,5 @@
         velocity="3.14"/>
       <dynamics damping="1.0" friction="1.0"/>
+      <initial_position>1.5708</initial_position>
     </joint>
     <link name="${prefix}link6">
@@ -194,10 +227,12 @@
         origin_rpy="0 0 0"/>
       <xacro:common_link_visual
-        mesh_filename="${end_tool_visual_filename}"
+        mesh_filename="${link6_visual}"
         origin_xyz="0 0 0"
         origin_rpy="0 0 0"
         material_name="${prefix}Silver" />
       <xacro:common_link_collision
-        mesh_filename="${end_tool_collision_filename}"
+        mesh_filename="${link6_collision}"
+        add_mesh_suffix="${add_mesh_suffix}"
+        other_mesh_suffix="${collison_mesh_suffix}"
         origin_xyz="0 0 0"
         origin_rpy="0 0 0" />
@@ -215,11 +250,276 @@
         velocity="3.14"/>
       <dynamics damping="1.0" friction="1.0"/>
-    </joint>
-    <!-- <link name="${prefix}link_eef" />
-    <joint name="${prefix}joint_eef" type="fixed">
+      <initial_position>0.0</initial_position>
+    </joint>
+  <!-- Gripper components -->
+  <joint name="${prefix}gripper_fix" type="fixed">
+    <parent link="${prefix}link6"/>
+    <child link="${prefix}xarm_gripper_base_link"/>
+    <origin rpy="0 0 0" xyz="0 0 0"/>
+  </joint>
+  <link name="${prefix}xarm_gripper_base_link">
+    <inertial>
+      <origin rpy="0 0 0" xyz="-0.00065489 -0.0018497 0.048028"/>
+      <mass value="0.54156"/>
+      <inertia ixx="0.00047106" ixy="3.9292E-07" ixz="2.6537E-06" iyy="0.00033072" iyz="-1.0975E-05" izz="0.00025642"/>
+    </inertial>
+    <visual>
+      <origin rpy="0 0 0" xyz="0 0 0"/>
+      <geometry>
+        <mesh filename="${mesh_path}/gripper/xarm/base_link.stl"/>
+      </geometry>
+      <material name="${prefix}White"/>
+    </visual>
+    <collision>
+      <origin rpy="0 0 0" xyz="0 0 0"/>
+      <geometry>
+        <mesh filename="${mesh_path}/gripper/xarm/base_link.stl"/>
+      </geometry>
+    </collision>
+  </link>
+  <link name="${prefix}left_outer_knuckle">
+    <inertial>
+      <origin rpy="0 0 0" xyz="2.9948E-14 0.021559 0.015181"/>
+      <mass value="0.033618"/>
+      <inertia ixx="1.9111E-05" ixy="-1.8803E-17" ixz="-1.1002E-17" iyy="6.6256E-06" iyz="-7.3008E-06" izz="1.3185E-05"/>
+    </inertial>
+    <visual>
+      <origin rpy="0 0 0" xyz="0 0 0"/>
+      <geometry>
+        <mesh filename="${mesh_path}/gripper/xarm/left_outer_knuckle.stl"/>
+      </geometry>
+      <material name="${prefix}Silver"/>
+    </visual>
+    <collision>
+      <origin rpy="0 0 0" xyz="0 0 0"/>
+      <geometry>
+        <mesh filename="${mesh_path}/gripper/xarm/left_outer_knuckle.stl"/>
+      </geometry>
+    </collision>
+  </link>
+  <xacro:if value="${lock_gripper}">
+    <joint name="${prefix}drive_joint" type="fixed">
+      <origin rpy="${driver_joint} 0 0" xyz="0 0.035 0.059098"/>
+      <parent link="${prefix}xarm_gripper_base_link"/>
+      <child  link="${prefix}left_outer_knuckle"/>
+    </joint>
+  </xacro:if>
+  <xacro:unless value="${lock_gripper}">
+    <joint name="${prefix}drive_joint" type="revolute">
+      <origin rpy="0 0 0" xyz="0 0.035 0.059098"/>
+      <parent link="${prefix}xarm_gripper_base_link"/>
+      <child  link="${prefix}left_outer_knuckle"/>
+      <axis xyz="1 0 0"/>
+      <limit effort="50" lower="0" upper="0.85" velocity="2"/>
+      <dynamics damping="1.0" friction="1.0"/>
+      <initial_position>0.0</initial_position>
+    </joint>
+  </xacro:unless>
+  <link name="${prefix}left_finger">
+    <inertial>
+      <origin rpy="0 0 0" xyz="-2.4536E-14 -0.016413 0.029258"/>
+      <mass value="0.048304"/>
+      <inertia ixx="1.7493E-05" ixy="-4.2156E-19" ixz="6.9164E-18" iyy="1.7225E-05" iyz="4.6433E-06" izz="5.1466E-06"/>
+    </inertial>
+    <visual>
+      <origin rpy="0 0 0" xyz="0 0 0"/>
+      <geometry>
+        <mesh filename="${mesh_path}/gripper/xarm/left_finger.stl"/>
+      </geometry>
+      <material name="${prefix}Silver"/>
+    </visual>
+    <collision>
+      <origin rpy="0 0 0" xyz="0 0 0"/>
+      <geometry>
+        <mesh filename="${mesh_path}/gripper/xarm/left_finger.stl"/>
+      </geometry>
+    </collision>
+  </link>
+  <xacro:if value="${lock_gripper}">
+    <joint name="${prefix}left_finger_joint" type="fixed">
+      <origin rpy="-${driver_joint} 0 0" xyz="0 0.035465 0.042039"/>
+      <parent link="${prefix}left_outer_knuckle"/>
+      <child link="${prefix}left_finger"/>
+    </joint>
+  </xacro:if>
+  <xacro:unless value="${lock_gripper}">
+    <joint name="${prefix}left_finger_joint" type="revolute">
+      <origin rpy="0 0 0" xyz="0 0.035465 0.042039"/>
+      <parent link="${prefix}left_outer_knuckle"/>
+      <child link="${prefix}left_finger"/>
+      <axis xyz="-1 0 0"/>
+      <limit effort="50" lower="0" upper="0.85" velocity="2"/>
+      <mimic joint="${prefix}drive_joint" multiplier="1" offset="0"/>
+      <dynamics damping="1.0" friction="1.0"/>
+    </joint>
+  </xacro:unless>
+  <link name="${prefix}left_inner_knuckle">
+    <inertial>
+      <origin rpy="0 0 0" xyz="1.86600784687907E-06 0.0220467847633621 0.0261334672830885"/>
+      <mass value="0.0230125781256706"/>
+      <inertia ixx="6.09490024271906E-06" ixy="6.06651326160071E-11" ixz="7.19102670500635E-11" iyy="6.01955084375188E-06" iyz="-2.75316812991721E-06" izz="5.07862004479903E-06"/>
+    </inertial>
+    <visual>
+      <origin rpy="0 0 0" xyz="0 0 0"/>
+      <geometry>
+        <mesh filename="${mesh_path}/gripper/xarm/left_inner_knuckle.stl"/>
+      </geometry>
+      <material name="${prefix}Silver"/>
+    </visual>
+    <collision>
+      <origin rpy="0 0 0" xyz="0 0 0"/>
+      <geometry>
+        <mesh filename="${mesh_path}/gripper/xarm/left_inner_knuckle.stl"/>
+      </geometry>
+    </collision>
+  </link>
+  <xacro:if value="${lock_gripper}">
+    <joint name="${prefix}left_inner_knuckle_joint" type="fixed">
+      <origin rpy="${driver_joint} 0 0" xyz="0 0.02 0.074098"/>
+      <parent link="${prefix}xarm_gripper_base_link"/>
+      <child link="${prefix}left_inner_knuckle"/>
+    </joint>
+  </xacro:if>
+  <xacro:unless value="${lock_gripper}">
+    <joint name="${prefix}left_inner_knuckle_joint" type="revolute">
+      <origin rpy="0 0 0" xyz="0 0.02 0.074098"/>
+      <parent link="${prefix}xarm_gripper_base_link"/>
+      <child link="${prefix}left_inner_knuckle"/>
+      <axis xyz="1 0 0"/>
+      <limit effort="50" lower="0" upper="0.85" velocity="2"/>
+      <mimic joint="${prefix}drive_joint" multiplier="1" offset="0"/>
+      <dynamics damping="1.0" friction="1.0"/>
+    </joint>
+  </xacro:unless>
+  <link name="${prefix}right_outer_knuckle">
+    <inertial>
+      <origin rpy="0 0 0" xyz="-3.1669E-14 -0.021559 0.015181"/>
+      <mass value="0.033618"/>
+      <inertia ixx="1.9111E-05" ixy="-1.8789E-17" ixz="1.0986E-17" iyy="6.6256E-06" iyz="7.3008E-06" izz="1.3185E-05"/>
+    </inertial>
+    <visual>
+      <origin rpy="0 0 0" xyz="0 0 0"/>
+      <geometry>
+        <mesh filename="${mesh_path}/gripper/xarm/right_outer_knuckle.stl"/>
+      </geometry>
+      <material name="${prefix}Silver"/>
+    </visual>
+    <collision>
+      <origin rpy="0 0 0" xyz="0 0 0"/>
+      <geometry>
+        <mesh filename="${mesh_path}/gripper/xarm/right_outer_knuckle.stl"/>
+      </geometry>
+    </collision>
+  </link>
+  <xacro:if value="${lock_gripper}">
+    <joint name="${prefix}right_outer_knuckle_joint" type="fixed">
+      <origin rpy="-${driver_joint} 0 0" xyz="0 -0.035 0.059098"/>
+      <parent link="${prefix}xarm_gripper_base_link"/>
+      <child link="${prefix}right_outer_knuckle"/>
+    </joint>
+  </xacro:if>
+  <xacro:unless value="${lock_gripper}">
+    <joint name="${prefix}right_outer_knuckle_joint" type="revolute">
+      <origin rpy="0 0 0" xyz="0 -0.035 0.059098"/>
+      <parent link="${prefix}xarm_gripper_base_link"/>
+      <child link="${prefix}right_outer_knuckle"/>
+      <axis xyz="-1 0 0"/>
+      <limit effort="50" lower="0" upper="0.85" velocity="2"/>
+      <mimic joint="${prefix}drive_joint" multiplier="1" offset="0"/>
+      <dynamics damping="1.0" friction="1.0"/>
+    </joint>
+  </xacro:unless>
+  <link name="${prefix}right_finger">
+    <inertial>
+      <origin rpy="0 0 0" xyz="2.5618E-14 0.016413 0.029258"/>
+      <mass value="0.048304"/>
+      <inertia ixx="1.7493E-05" ixy="-5.0014E-19" ixz="-7.5079E-18" iyy="1.7225E-05" iyz="-4.6435E-06" izz="5.1466E-06"/>
+    </inertial>
+    <visual>
+      <origin rpy="0 0 0" xyz="0 0 0"/>
+      <geometry>
+        <mesh filename="${mesh_path}/gripper/xarm/right_finger.stl"/>
+      </geometry>
+      <material name="${prefix}Silver"/>
+    </visual>
+    <collision>
+      <origin rpy="0 0 0" xyz="0 0 0"/>
+      <geometry>
+        <mesh filename="${mesh_path}/gripper/xarm/right_finger.stl"/>
+      </geometry>
+    </collision>
+  </link>
+  <xacro:if value="${lock_gripper}">
+    <joint name="${prefix}right_finger_joint" type="fixed">
+      <origin rpy="${driver_joint} 0 0" xyz="0 -0.035465 0.042039"/>
+      <parent link="${prefix}right_outer_knuckle"/>
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
File: xarm_description/urdf/xarm6/xarm6_robot_macro.xacro (robot description, xacro)
@@ -13,5 +13,5 @@
     baud_checkset:='true'
     default_gripper_baud:=2000000
-    model1300:=false
+    model_num:=0
     inertial_params_filename:=''
     kinematics_params_filename:=''
@@ -22,5 +22,5 @@
       <xacro:include filename="$(find xarm_description)/urdf/xarm6/xarm6.ros2_control.xacro" />
     </xacro:if>
-    <xacro:include filename="$(find xarm_description)/urdf/xarm6/xarm6.urdf.xacro" />
+    <xacro:include filename="$(find xarm_description)/urdf/xarm6/xarm6_stick.urdf.xacro" />
     <xacro:include filename="$(find xarm_description)/urdf/xarm6/xarm6.transmission.xacro" />
     <xacro:include filename="$(find xarm_description)/urdf/xarm6/xarm6.gazebo.xacro" />
@@ -47,5 +47,5 @@
         joint5_lower_limit="${-1.69297}" joint5_upper_limit="${pi*0.99}"
         joint6_lower_limit="${-pi*0.99}" joint6_upper_limit="${pi*0.99}"
-        model1300="${model1300}"
+        model_num="${model_num}"
         inertial_params_filename="${inertial_params_filename}"
         kinematics_params_filename="${kinematics_params_filename}"
@@ -60,5 +60,5 @@
           baud_checkset="${baud_checkset}" default_gripper_baud="${default_gripper_baud}" />
       </xacro:if>
-      <xacro:xarm6_urdf prefix="${prefix}" model1300="${model1300}"
+      <xacro:xarm6_urdf prefix="${prefix}" model_num="${model_num}"
         inertial_params_filename="${inertial_params_filename}"
         kinematics_params_filename="${kinematics_params_filename}"
@@ -67,4 +67,11 @@
     <xacro:xarm6_transmission prefix="${prefix}" hard_interface="${hard_interface}" />
     <xacro:xarm6_gazebo prefix="${prefix}" />
+    <xacro:property name="M_PI" value="3.1415926535897931" />
+    <link name="wrist_camera_link" />
+    <joint name="wrist_camera_link_joint" type="fixed">
+      <parent link="${prefix}link_eef" />
+      <child link="wrist_camera_link" />
+      <origin xyz="0.06746 -0.0575 0.0237" rpy="${M_PI} ${-M_PI/2} 0" />
+    </joint>
   </xacro:macro>
 </robot>

File: xarm_description/urdf/xarm_device.urdf.xacro (robot description, xacro)
@@ -1,4 +1,4 @@
 <?xml version='1.0' encoding='utf-8'?>
-<robot xmlns:xacro="http://ros.org/wiki/xacro" name="UF_ROBOT">
+<robot xmlns:xacro="http://ros.org/wiki/xacro" name="xarm_device">
   <!-- macro for having property with the same name/value as an argument -->
   <xacro:macro name="define_arg_property" params="prop_name default">
@@ -7,5 +7,5 @@
   </xacro:macro>
   <xacro:arg name="prefix" default=""/>
-  <xacro:arg name="hw_ns" default="xarm"/>
+  <xacro:arg name="hw_ns" default=""/>
   <xacro:arg name="ros2_control_plugin" default="uf_robot_hardware/UFRobotSystemHardware"/>
   <xacro:arg name="ros2_control_params" default=""/>
@@ -58,5 +58,5 @@
     baud_checkset="${robot_spec['baud_checkset']}"
     default_gripper_baud="${robot_spec['default_gripper_baud']}"
-    model1300="${robot_spec['model1300']}"
+    model_num="${robot_spec['model_num']}"
     robot_sn="${robot_spec['robot_sn']}"
     limited="${robot_spec['limited']}"
@@ -66,4 +66,5 @@
     attach_xyz="${robot_spec['attach_xyz']}"
     attach_rpy="${robot_spec['attach_rpy']}"
+    create_attach_link="${robot_spec['create_attach_link']}"
     mesh_suffix="${robot_spec['mesh_suffix']}"
     kinematics_suffix="${robot_spec['kinematics_suffix']}"
