Commit message: Cleanup with latest -- using OI-MPPI
* Robot position

* _robot_joint_state.launch.py fixed

* moveit

* fix control launch

* propagate changes to gazebo

* Incorporating moveit in xarm6

* Moveit in besides_table world

* Incorporating moveit

* trying to revert namespacing

* works without namespace

* make single robot planning work

* Added camera and ros_gz_bridge node

* minor

* minor

* correct camera orientation

* Adding gripper

* minor

* octomap

* Fix TF tree (#10)

* TF tree now connected, but robot falls over

* robot doesn't fall down now, but sim is slow

* use keti_gz_utils create instead

* remove the 'heavy' link

---------

Co-authored-by: brian <brian@erl-brian>

* world_table.sdf changed

* Added [200~# Software License Agreement (BSD License)

* use a simple timer for the moment

* minor

* updated real robot_ip

* Gazebo velocity controller

* Velocity controller

* Controller specifing robot description

* use different kinematics yaml between sim and real

* Offset handling

* add user/xarm6_kinematics_sim.yaml

* minor

* [MPPI-Isaac] Integrated code into xarm_ros2 mppi branch.

* [Orient test] Match the limitation of joint velocity

* [Velocity Controller] Integrated

* [Gripper] Working on gripper

* [Fixed Gripper]

* Controller

* minor

* sanity check of orientation

* [Rviz] Finished MPPI visualization.

* Lab setup issue

* [Dev-mode] Joint state publishing frequency is 100 Hz

* add stick

* set up for sim

* update stick with isaac

* [Collision Geometry] Adding wrist camera and collision step

* wrist camera version

* update wrist camera position (#13)

Co-authored-by: Dwait Bhatt <dhbhatt@ucsd.edu>

---------

Co-authored-by: NikolaRaicevic <nikolar047@gmail.com>
Co-authored-by: Brian Lee <brian@UTS040524>
Co-authored-by: brian <brian@erl-brian>
Co-authored-by: Niyas-A <niyasttshr33@gmail.com>
Co-authored-by: Dwait Bhatt <dhbhatt@ucsd.edu>
Co-authored-by: NikolaRaicevic2001 <nmarinosraitsevits@ucsd.edu>
Co-authored-by: ticotico410 <ycb04106438which pip.com>

File: xarm_description/urdf/xarm_device_macro.xacro (robot description, xacro)
@@ -3,5 +3,5 @@
   <xacro:macro name="xarm_device" params="
     prefix:=''
-    hw_ns:='xarm'
+    hw_ns:=''
     limited:=false
     effort_control:=false
@@ -37,5 +37,5 @@
     baud_checkset:=true
     default_gripper_baud:=2000000
-    model1300:=false
+    model_num:=0
     robot_sn:=''
     mesh_suffix:='stl'
@@ -60,16 +60,18 @@
     <!-- include common.link.xacro -->
     <xacro:include filename="$(find xarm_description)/urdf/common/common.link.xacro" />
-    <xacro:parse_link_inertial_filename dof="${dof}" robot_type="${robot_type}" robot_sn="${robot_sn}" model1300="${model1300}" />
+    <xacro:parse_link_inertial_filename dof="${dof}" robot_type="${robot_type}" robot_sn="${robot_sn}" model_num="${model_num}" />
     <xacro:property name="inertial_params_filename" value="${scope_parent_inertial_params_filename}"/>
-    <xacro:property name="new_model1300" value="${scope_parent_model1300}"/>
+    <xacro:property name="new_model_num" value="${scope_parent_model_num}"/>
     <!-- add one world link if no 'attach_to' specified  -->
-    <xacro:if value="${attach_to == 'world' and create_attach_link}">
-      <link name="world" />
-    </xacro:if>
-    <joint name="${prefix}world_joint" type="fixed">
-      <parent link="${attach_to}" />
-      <child link="${prefix}link_base" />
-      <origin xyz="${attach_xyz}" rpy="${attach_rpy}" />
-    </joint>
+    <xacro:if value="${attach_to != ''}">
+      <xacro:if value="${create_attach_link}">
+        <link name="${attach_to}" />
+      </xacro:if>
+      <joint name="${prefix}world_joint" type="fixed">
+        <parent link="${attach_to}" />
+        <child link="${prefix}link_base" />
+        <origin xyz="${attach_xyz}" rpy="${attach_rpy}" />
+      </joint>
+    </xacro:if>
     <xacro:if value="${effort_control}">
       <xacro:property name="hard_interface" value="EffortJointInterface" />
@@ -125,5 +127,5 @@
           baud_checkset="${baud_checkset}"
           default_gripper_baud="${default_gripper_baud}"
-          model1300="${new_model1300}"
+          model_num="${new_model_num}"
           inertial_params_filename="${inertial_params_filename}"
           kinematics_params_filename="${kinematics_params_filename}"
@@ -157,5 +159,5 @@
           baud_checkset="${baud_checkset}"
           default_gripper_baud="${default_gripper_baud}"
-          model1300="${new_model1300}"
+          model_num="${model_num}"
           inertial_params_filename="${inertial_params_filename}"
           kinematics_params_filename="${kinematics_params_filename}"
@@ -176,5 +178,5 @@
           baud_checkset="${baud_checkset}"
           default_gripper_baud="${default_gripper_baud}"
-          model1300="${new_model1300}"
+          model_num="${new_model_num}"
           inertial_params_filename="${inertial_params_filename}"
           kinematics_params_filename="${kinematics_params_filename}"
@@ -193,5 +195,5 @@
           baud_checkset="${baud_checkset}"
           default_gripper_baud="${default_gripper_baud}"
-          model1300="${new_model1300}"
+          model_num="${new_model_num}"
           inertial_params_filename="${inertial_params_filename}"
           kinematics_params_filename="${kinematics_params_filename}"
@@ -205,10 +207,24 @@
       <xacro:d435i_urdf prefix="${prefix}" add_d435i_links="${add_d435i_links}" />
       <xacro:if value="${add_d435i_links}">
-        <xacro:include filename="$(find xarm_description)/urdf/camera/realsense.gazebo.xacro" />
-        <xacro:realsense_gazebo prefix="${prefix}" />
+        <xacro:if value="${ros2_control_plugin == 'ign_ros2_control/IgnitionSystem'}">
+          <xacro:include filename="$(find xarm_description)/urdf/camera/realsense.gz.xacro" />
+          <xacro:realsense_gz prefix="${prefix}" />
+        </xacro:if>
+        <xacro:unless value="${ros2_control_plugin == 'ign_ros2_control/IgnitionSystem'}">
+          <xacro:include filename="$(find xarm_description)/urdf/camera/realsense.gazebo.xacro" />
+          <xacro:realsense_gazebo prefix="${prefix}" />
+        </xacro:unless>
       </xacro:if>
     </xacro:if>
     <xacro:unless value="${add_realsense_d435i}">
-      <link name="${prefix}link_eef"/>
+      <link name="${prefix}link_eef">
+        <inertial>
+          <origin xyz="0 0 0" rpy="0 0 0" />
+          <mass value="0.001" />
+          <inertia
+            ixx="0.000001" ixy="0.0" ixz="0.0"
+            iyy="0.000001" iyz="0.0" izz="0.000001" />
+        </inertial>
+      </link>
     </xacro:unless>
     <joint name="${prefix}joint_eef" type="fixed">
@@ -284,4 +300,18 @@
     </xacro:if>
     <xacro:device_macro_end />
+    <gazebo>
+        <plugin filename="ignition-gazebo-pose-publisher-system" name="gz::sim::systems::PosePublisher">
+            <publish_link_pose>false</publish_link_pose>
+            <publish_visual_pose>false</publish_visual_pose>
+            <publish_collision_pose>false</publish_collision_pose>
+            <publish_sensor_pose>false</publish_sensor_pose>
+            <publish_model_pose>true</publish_model_pose>
+            <publish_nested_model_pose>true</publish_nested_model_pose>
+            <use_pose_vector_msg>true</use_pose_vector_msg>
+            <update_frequency>10</update_frequency>
+            <static_publisher>false</static_publisher>
+            <static_update_frequency>10</static_update_frequency>
+        </plugin>
+    </gazebo>
   </xacro:macro>
 </robot>

Commit message: add cbf sim

File: xarm_description/urdf/xarm6/xarm6.ros2_control.xacro (robot description, xacro)
@@ -13,5 +13,9 @@
     joint6_lower_limit:=${-10*pi}  joint6_upper_limit:=${10*pi}">
     <!-- Define initial joint position -->
-    <xacro:property name="init_joint_pos" value="${[0.0, -0.78, -0.78, 0.0, 1.5708, 0.0]}" />
+    <!-- Arm starts higher than the canonical "ready" pose so the stick EE
+         has 30+cm of clearance above the table for the CBF demo. joint2/3
+         bend less, joint5 still pitches the wrist down so the camera looks
+         straight at the table. -->
+    <xacro:property name="init_joint_pos" value="${[0.0, -0.30, -0.30, 0.0, 0.6, 0.0]}" />
     <ros2_control name="${prefix}${ros2_control_plugin}" type="system">
       <hardware>
