Commit message: Lab setup issue

File: xarm_description/urdf/gripper/bio_gripper.urdf.xacro (robot description, xacro)
@@ -78,5 +78,13 @@
       <limit lower="0" upper="0.04" effort="2.0" velocity="0.1" />
     </joint>
-    <link name="${prefix}link_tcp" />
+    <link name="${prefix}link_tcp">
+      <inertial>
+        <origin xyz="0 0 0" rpy="0 0 0" />
+        <mass value="0.001" />
+        <inertia
+          ixx="0.000001" ixy="0.0" ixz="0.0"
+          iyy="0.000001" iyz="0.0" izz="0.000001" />
+      </inertial>
+    </link>
     <joint name="${prefix}joint_tcp" type="fixed">
       <origin xyz="0.135 0 0.055" rpy="0 0 0" />

File: xarm_description/urdf/gripper/lite_gripper.urdf.xacro (robot description, xacro)
@@ -27,5 +27,13 @@
         origin_rpy="0 0 0" />
     </link>
-    <link name="${prefix}link_tcp" />
+    <link name="${prefix}link_tcp">
+      <inertial>
+        <origin xyz="0 0 0" rpy="0 0 0" />
+        <mass value="0.001" />
+        <inertia
+          ixx="0.000001" ixy="0.0" ixz="0.0"
+          iyy="0.000001" iyz="0.0" izz="0.000001" />
+      </inertial>
+    </link>
     <joint name="${prefix}joint_tcp" type="fixed">
       <origin xyz="0 0 0.0836" rpy="0 0 0" />

File: xarm_description/urdf/gripper/xarm_gripper.urdf.xacro (robot description, xacro)
@@ -182,5 +182,13 @@
       <mimic joint="${prefix}drive_joint" multiplier="1" offset="0" />
     </joint>
-    <link name="${prefix}link_tcp" />
+    <link name="${prefix}link_tcp">
+      <inertial>
+        <origin xyz="0 0 0" rpy="0 0 0" />
+        <mass value="0.001" />
+        <inertia
+          ixx="0.000001" ixy="0.0" ixz="0.0"
+          iyy="0.000001" iyz="0.0" izz="0.000001" />
+      </inertial>
+    </link>
     <joint name="${prefix}joint_tcp" type="fixed">
       <origin xyz="0 0 0.172" rpy="0 0 0" />

File: xarm_description/urdf/other/other_geometry.urdf.xacro (robot description, xacro)
@@ -98,5 +98,13 @@
       </collision>
     </link>
-    <link name="${prefix}link_tcp" />
+    <link name="${prefix}link_tcp">
+      <inertial>
+        <origin xyz="0 0 0" rpy="0 0 0" />
+        <mass value="0.001" />
+        <inertia
+          ixx="0.000001" ixy="0.0" ixz="0.0"
+          iyy="0.000001" iyz="0.0" izz="0.000001" />
+      </inertial>
+    </link>
     <joint name="${prefix}joint_tcp" type="fixed">
       <origin xyz="${_tcp_xyz}" rpy="${_tcp_rpy}" />

File: xarm_description/urdf/vacuum_gripper/xarm_vacuum_gripper.urdf.xacro (robot description, xacro)
@@ -27,5 +27,13 @@
         origin_rpy="0 0 0" />
     </link>
-    <link name="${prefix}link_tcp" />
+    <link name="${prefix}link_tcp">
+      <inertial>
+        <origin xyz="0 0 0" rpy="0 0 0" />
+        <mass value="0.001" />
+        <inertia
+          ixx="0.000001" ixy="0.0" ixz="0.0"
+          iyy="0.000001" iyz="0.0" izz="0.000001" />
+      </inertial>
+    </link>
     <joint name="${prefix}joint_tcp" type="fixed">
       <origin xyz="0 0 0.126" rpy="0 0 0" />

File: xarm_description/urdf/xarm6/xarm6.urdf.xacro (robot description, xacro)
@@ -508,4 +508,11 @@
   <!-- Gripper ee_tip -->
   <link name="${prefix}gripper_ee_tip">
+    <inertial>
+      <origin xyz="0 0 0" rpy="0 0 0" />
+      <mass value="0.001" />
+      <inertia
+        ixx="0.000001" ixy="0.0" ixz="0.0"
+        iyy="0.000001" iyz="0.0" izz="0.000001" />
+    </inertial>
   </link>
   <joint name="${prefix}gripper_ee_tip_joint" type="fixed">

File: xarm_description/urdf/xarm_device_macro.xacro (robot description, xacro)
@@ -212,5 +212,13 @@
     </xacro:if>
     <xacro:unless value="${add_realsense_d435i}">
-      <link name="${prefix}link_eef"/>
+      <link name="${prefix}link_eef">
+        <inertial>
+          <origin xyz="0 0 0" rpy="0 0 0" />
+          <mass value="0.001" />
+          <inertia
+            ixx="0.000001" ixy="0.0" ixz="0.0"
+            iyy="0.000001" iyz="0.0" izz="0.000001" />
+        </inertial>
+      </link>
     </xacro:unless>
     <joint name="${prefix}joint_eef" type="fixed">
