Commit message: wrist camera sim

File: xarm_description/urdf/camera/realsense.gz.xacro (robot description, xacro)
@@ -14,6 +14,6 @@
   <xacro:macro name="realsense_gz" params="
     prefix:=''
-    camera_name:='camera'
-    update_rate:=30
+    camera_name:='wrist_camera'
+    update_rate:=10
     image_width:=1280
     image_height:=720
@@ -42,5 +42,5 @@
         <gz_frame_id>${prefix}camera_depth_frame</gz_frame_id>
         <ignition_frame_id>${prefix}camera_depth_frame</ignition_frame_id>
-        <topic>${prefix}${camera_name}/depth</topic>
+        <topic>${prefix}${camera_name}/depth/image_rect_raw</topic>
       </sensor>
     </gazebo>
@@ -70,5 +70,5 @@
         <gz_frame_id>${prefix}camera_color_frame</gz_frame_id>
         <ignition_frame_id>${prefix}camera_color_frame</ignition_frame_id>
-        <topic>${prefix}${camera_name}/color</topic>
+        <topic>${prefix}${camera_name}/color/image_raw</topic>
       </sensor>
     </gazebo>

File: xarm_description/urdf/camera/realsense_d435i.urdf.xacro (robot description, xacro)
@@ -5,13 +5,26 @@
     <xacro:property name="M_PI" value="3.1415926535897931" />
     <link name="${prefix}link_eef">
-      <xacro:common_link_visual
-        mesh_filename="camera/realsense/visual/d435_with_cam_stand"
-        origin_xyz="0 0 0"
-        origin_rpy="0 0 0"
-        material_name="${prefix}Silver" />
-      <xacro:common_link_collision
-        mesh_filename="camera/realsense/collision/d435_with_cam_stand"
-        origin_xyz="0 0 0"
-        origin_rpy="0 0 0" />
+      <!-- Bare d435 body, no cam-stand "stick". The mesh's local origin is
+           the camera optical center; the camera_link joint origin below
+           still expresses optics relative to the wrist flange. -->
+      <visual>
+        <origin xyz="0 0 0" rpy="0 0 0"/>
+        <geometry>
+          <mesh filename="${mesh_path}/camera/realsense/visual/d435.dae"/>
+        </geometry>
+      </visual>
+      <collision>
+        <origin xyz="0 0 0" rpy="0 0 0"/>
+        <geometry>
+          <box size="0.025 0.090 0.025"/>
+        </geometry>
+      </collision>
+      <inertial>
+        <origin xyz="0 0 0" rpy="0 0 0"/>
+        <mass value="0.072"/>
+        <inertia
+          ixx="0.0001" ixy="0.0" ixz="0.0"
+          iyy="0.0001" iyz="0.0" izz="0.0001"/>
+      </inertial>
     </link>
     <xacro:if value="${add_d435i_links}">
